File: BulkyMIDI-32 Module/BulkyMIDI-32 Module.kicad_pcb (KiCad board)
At the start: 2 copper layers, 100 x 100 mm, 24 parts, among them IC1 1.3_OLED, J1 DC IN, J2 DIN5_MIDI, J3 DIN5_MIDI, J4 Faceplate, M1 Mounting, M2 Mounting, M3 Mounting, M4 Mounting, SW1 SYNTH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

Commit message: Routed tracks
Parts:
- removed D3: POWER, LEDs:LED_D5.0mm
- removed R7: 330, Resistors_THT:R_Axial_DIN0207_L6.3mm_D2.5mm_P10.16mm_Horizontal
- removed REF** (x2): Symbol_Barrel_Polarity, Symbols:Symbol_Barrel_Polarity
- added A2: GY-PCM5102, BulkyMIDI-32:GY-PCM5102, F.Cu at (104.9, 63.2)
- added C3: 100nF, Capacitor_THT:C_Rect_L7.0mm_W2.0mm_P5.00mm, F.Cu at (120.0, 77.5)
- added C4: 100nF, Capacitor_THT:C_Rect_L7.0mm_W2.0mm_P5.00mm, F.Cu at (109.2, 73.7)
- added C5: 100uF, Capacitor_THT:CP_Radial_D6.3mm_P2.50mm, F.Cu at (114.3, 74.9)
- added C6: 470uF, Capacitor_THT:CP_Radial_D8.0mm_P3.50mm, F.Cu at (83.2, 73.7)
- added D1: 1N4148, Diode_THT:D_DO-35_SOD27_P7.62mm_Horizontal, F.Cu at (132.7, 83.8)
- added ENC1: KY-040, Connector_PinHeader_2.54mm:PinHeader_1x05_P2.54mm_Horizontal, F.Cu at (159.4, 123.2)
- added J5: MIDI Thru Jack, Connector_PinHeader_2.54mm:PinHeader_1x05_P2.54mm_Horizontal, F.Cu at (159.4, 96.5)
- added J6: Serial, Connector_PinHeader_2.54mm:PinHeader_1x04_P2.54mm_Horizontal, F.Cu at (159.4, 111.1)
- added JP3: SW4_SEL, Jumper:SolderJumper-3_P1.3mm_Open_RoundedPad1.0x1.5mm, B.Cu at (142.2, 143.5)
- added R1: 220, Resistor_THT:R_Axial_DIN0207_L6.3mm_D2.5mm_P10.16mm_Horizontal, F.Cu at (167.0, 62.9)
- added R2: 220, Resistor_THT:R_Axial_DIN0207_L6.3mm_D2.5mm_P10.16mm_Horizontal, F.Cu at (146.1, 76.2)
- added R3: 1k, Resistor_THT:R_Axial_DIN0207_L6.3mm_D2.5mm_P10.16mm_Horizontal, F.Cu at (146.1, 80.0)
- added R4: 220, Resistor_THT:R_Axial_DIN0207_L6.3mm_D2.5mm_P10.16mm_Horizontal, F.Cu at (146.1, 83.8)
- added R5: 220, Resistor_THT:R_Axial_DIN0207_L6.3mm_D2.5mm_P10.16mm_Horizontal, F.Cu at (149.2, 96.5)
- added SYM1: DC_5V, BulkyMIDI-32:PWR_Specification, F.Cu at (83.2, 56.5)
- added U2: H11L1M, Package_DIP:DIP-6_W7.62mm, F.Cu at (124.0, 83.8)
- A1: value Raspberry PI -> Raspberry PI 3B
- C1: footprint Capacitors_THT:C_Disc_D4.7mm_W2.5mm_P5.00mm -> Capacitor_THT:C_Rect_L7.0mm_W2.0mm_P5.00mm
- IC1: value 1.3_OLED -> OLED
- J2: value DIN5_MIDI -> MIDI OUT
- J3: value DIN5_MIDI -> MIDI IN
- J4: footprint Pin_Headers:Pin_Header_Straight_1x04_Pitch2.54mm -> Connector_PinSocket_2.54mm:PinSocket_1x10_P2.54mm_Vertical
- JP1, JP2: footprint wire_pads:OLED_SEL -> Jumper:SolderJumper-3_P1.3mm_Open_RoundedPad1.0x1.5mm; moved to B.Cu
- R6: value 330 -> 220; footprint Resistors_THT:R_Axial_DIN0207_L6.3mm_D2.5mm_P10.16mm_Horizontal -> Resistor_THT:R_Axial_DIN0207_L6.3mm_D2.5mm_P10.16mm_Horizontal
- SW1, SW2, SW3, SW4: footprint Buttons_Switches_THT:SW_Tactile_SPST_Angled_PTS645Vx39-2LFS -> Button_Switch_THT:SW_Tactile_SPST_Angled_PTS645Vx39-2LFS
- U1: footprint Housings_DIP:DIP-14_W7.62mm_LongPads -> Package_DIP:DIP-14_W7.62mm
- moved R6 51.5 mm to (153.0, 106.7)
- moved C1 20.3 mm to (149.2, 77.5)
- moved U1 19.7 mm to (152.4, 83.8)
- moved REF*** 9.44 mm to (135.4, 123.1)
- moved JP1 5.68 mm to (101.0, 149.9), turned to 180 degrees
- moved JP2 5.68 mm to (95.9, 149.9), turned to 180 degrees
- moved J1 1.58 mm to (83.2, 68.6)
Connections:
- A1 pad 10: Net-(A1-Pad10) -> RX_TTL
- A1 pad 11: RPI_CLK_OUT -> SW_SYNTH
- A1 pad 12: RPI_DATA_OUT -> I2S_BCLK
- A1 pad 13: SW1 -> SW_ROM
- A1 pad 15: SW2 -> SW_DOWN
- A1 pad 16: SW3 -> SW_UP
- A1 pad 17: Net-(A1-Pad17) -> +3V3
- A1 pad 18: RPI_ATN -> (no net)
- A1 pad 19: Net-(A1-Pad19) -> (no net)
- A1 pad 21: Net-(A1-Pad21) -> (no net)
- A1 pad 22: RPI_DATA_IN -> (no net)
- A1 pad 23: Net-(A1-Pad23) -> (no net)
- A1 pad 24: Net-(A1-Pad24) -> (no net)
- A1 pad 26: Net-(A1-Pad26) -> (no net)
- A1 pad 27: Net-(A1-Pad27) -> (no net)
- A1 pad 28: Net-(A1-Pad28) -> (no net)
- A1 pad 29: SW5 -> (no net)
- A1 pad 31: Net-(A1-Pad31) -> (no net)
- A1 pad 32: Net-(A1-Pad32) -> (no net)
- A1 pad 33: Net-(A1-Pad33) -> (no net)
- A1 pad 35: Net-(A1-Pad35) -> I2S_LRCLK
- A1 pad 36: RPI_LED -> (no net)
- A1 pad 37: RPI_CLK_IN -> (no net)
- A1 pad 38: RPI_RST -> (no net)
- A1 pad 4: Net-(A1-Pad4) -> +5V
- A1 pad 40: Net-(A1-Pad40) -> I2S_DATA
- A1 pad 7: SW4 -> SW_ENC
- A1 pad 8: Net-(A1-Pad8) -> TX_TTL
- J2 pad 1: Net-(J2-Pad1) -> (no net)
- J2 pad 3: C64_ATN -> (no net)
- J2 pad 4: C64_CLK -> Net-(J2-Pad4)
- J2 pad 5: C64_DATA -> Net-(J2-Pad5)
- J3 pad 1: Net-(J3-Pad1) -> (no net)
- J3 pad 2: GND -> (no net)
- J3 pad 3: C64_ATN -> (no net)
- J3 pad 4: C64_CLK -> Net-(J3-Pad4)
- J3 pad 5: C64_DATA -> Net-(D1-Pad2)
- J4 pad 1: GND -> +3V3
- J4 pad 2: +3V3 -> I2C_SCL
- J4 pad 3: I2C_SCL -> I2C_SDA
- J4 pad 4: I2C_SDA -> GND
- R6 pad 2: +3V3 -> Net-(R6-Pad2)
- SW1 pad 2: SW2 -> SW_SYNTH
- SW2 pad 2: SW3 -> SW_ROM
- SW3 pad 2: SW5 -> SW_DOWN
- SW4 pad 2: SW4 -> Net-(JP3-Pad2)
- U1 pad 1: RPI_DATA_OUT -> TX_TTL
- U1 pad 10: Net-(IC2-Pad10) -> (no net)
- U1 pad 11: Net-(IC2-Pad11) -> GND
- U1 pad 12: Net-(IC2-Pad12) -> (no net)
- U1 pad 13: Net-(IC2-Pad13) -> GND
- U1 pad 2: C64_DATA -> Net-(U1-Pad2)
- U1 pad 3: RPI_CLK_OUT -> Net-(U1-Pad2)
- U1 pad 4: C64_CLK -> Net-(R1-Pad2)
- U1 pad 5: Net-(IC2-Pad5) -> RX_TTL
- U1 pad 6: Net-(IC2-Pad6) -> Net-(U1-Pad6)
- U1 pad 8: Net-(IC2-Pad8) -> Net-(R6-Pad2)
- U1 pad 9: Net-(IC2-Pad9) -> Net-(U1-Pad6)
Routing:
- net +3V3: track 10.7 -> 279.0 mm, vias 0 -> 6
- net I2C_SDA: track 0.00 -> 214.2 mm, vias 0 -> 5
- net I2C_SCL: track 0.00 -> 214.0 mm, vias 0 -> 5
- net SW_DOWN: track 0.00 -> 211.2 mm, vias 0 -> 1
- net SW_ENC: track 0.00 -> 209.0 mm, vias 0 -> 4
- net SW_UP: track 0.00 -> 205.8 mm, vias 0 -> 4
- net SW_SYNTH: track 0.00 -> 196.9 mm, vias 0 -> 3
- net SW_ROM: track 0.00 -> 196.5 mm, vias 0 -> 4
- net +5V: track 0.00 -> 173.2 mm
- net RX_TTL: track 0.00 -> 87.0 mm, vias 0 -> 4
- net TX_TTL: track 0.00 -> 44.5 mm, vias 0 -> 1
- net I2S_BCLK: track 0.00 -> 44.3 mm, vias 0 -> 2
- net I2S_DATA: track 0.00 -> 38.2 mm
- net Net-(R6-Pad2): track 0.00 -> 37.2 mm
- net I2S_LRCLK: track 0.00 -> 30.8 mm
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Other:
- net class Power: clearance 0.381 -> 0.2
- board text removed: "+"
- board text removed: "-"
- board text removed: "Disk dimensions: 133.7mm PCB dimensions: 97,79mm Scale factor: 0.73"

Commit message: Added simple logo
Parts:
- removed the REF*** at (135.4, 123.1)
- added G***: LOGO, artwork:BulkyMIDI-32, B.Cu at (128.9, 115.6)
- added G***: LOGO, artwork:BulkyMIDI-32, F.Cu at (128.9, 115.6)
- added REF***: KiCad-Logo2_6mm_SilkScreen, Symbols:KiCad-Logo2_6mm_SilkScreen, B.Cu at (133.3, 129.5)
- added REF***: KiCad-Logo2_6mm_SilkScreen, Symbols:KiCad-Logo2_6mm_SilkScreen, F.Cu at (125.1, 129.5)
Routing:
- net RX_TTL: track 87.0 -> 84.3 mm
