File: BulkyMIDI-32 Faceplate/BulkyMIDI-32 Faceplate.kicad_pcb (KiCad board)
At the start: 2 copper layers, 100 x 100 mm, 9 parts, among them J4 Faceplate, M1 Mounting, M2 Mounting, M3 Mounting, M4 Mounting, SW1 SYNTH, SW4 VOL_UP

Commit message: Gerber export
Other:
- rule pad_to_mask_clearance: 0.2 -> 0

Commit message: Fixed faceplate buttons
Parts:
- added G***: LOGO, artwork:BulkyMIDI-32, B.Cu at (120.2, 104.6)
- added G***: LOGO, artwork:BulkyMIDI-32, F.Cu at (120.2, 104.6)
Connections:
- J4 pad 4: (no net) -> GND
Other:
- board text added: "BulkyMIDI-32 Faceplate (rev. B) github.com/tebl"
- board text removed: "BulkyMIDI-32 Faceplate (rev. A) github.com/tebl"
