File: BulkyMIDI-32 Faceplate/BulkyMIDI-32 Faceplate.sch (KiCad schematic (older format))
At the start: 7 parts, among them J4 Faceplate, M1 Mounting, M2 Mounting, M3 Mounting, M4 Mounting, SW1 SYNTH, SW4 VOL_UP

Commit message: Fixed faceplate buttons
Parts:
- J4: symbol BulkyMIDI:Conn_Faceplate -> BulkyMIDI:Conn_Faceplate_Male
Connections:
- net GND: now also J4.4 (Pin_4)
Changed lines of the file:
@@
 $EndComp
 $Comp
-L BulkyMIDI:Conn_Faceplate J4
+L BulkyMIDI:Conn_Faceplate_Male J4
 U 1 1 5F3B6F1D
 P 7025 3650
@@
 Wire Wire Line
 	6750 3850 6825 3850
+$Comp
+L power:GND #PWR0101
+U 1 1 6201A43A
+P 6175 3625
+F 0 "#PWR0101" H 6175 3375 50  0001 C CNN
+F 1 "GND" H 6175 3475 50  0000 C CNN
+F 2 "" H 6175 3625 50  0001 C CNN
+F 3 "" H 6175 3625 50  0001 C CNN
+	1    6175 3625
+	-1   0    0    -1
+$EndComp
+Wire Wire Line
+	6825 3550 6175 3550
+Wire Wire Line
+	6175 3550 6175 3625
 $EndSCHEMATC
