File: adapters/Vertical Rotary Encoder/Vertical Rotary Encoder.kicad_pcb (KiCad board)
At the start: 2 copper layers, 19.1 x 23.2 mm, 4 parts, among them J1 Conn_01x04

Commit message: Changed default setting to match expected direction
Connections:
- JP1 pad 1: /A -> /B
- JP1 pad 3: /B -> /A
- JP2 pad 1: /B -> /A
- JP2 pad 3: /A -> /B
Routing:
- net /A: track 14.7 -> 10.3 mm
- net /B: track 10.6 -> 14.7 mm
- net DAT: track 17.9 -> 17.0 mm
