File: adapters/BulkyMIDI-32 Amiga/BulkyMIDI-32 Amiga.sch (KiCad schematic (older format))
At the start: 23 parts, among them J1 DB25_Female, J2 MIDI OUT, J3 MIDI IN, M1 Mounting, M2 Mounting, U1 6N138, U2 LM7805_TO220, U3 74LS00, U4 MAX232

Commit message: Specify correct MAX232A variant
Parts:
- U4: value MAX232 -> MAX232A
Changed lines of the file:
@@
 P 2850 5875
 F 0 "U4" H 2850 6325 50  0000 C CNN
-F 1 "MAX232" H 2850 6225 50  0000 C CNN
+F 1 "MAX232A" H 2850 6225 50  0000 C CNN
 F 2 "Package_DIP:DIP-16_W7.62mm_Socket_LongPads" H 2900 4825 50  0001 L CNN
 F 3 "http://www.ti.com/lit/ds/symlink/max232.pdf" H 2850 5975 50  0001 C CNN
