File: adapters/BulkyMIDI-32 Amiga IDC/BulkyMIDI-32 Amiga IDC.sch (KiCad schematic (older format))
At the start: 25 parts, among them J1 Amiga Serial, J2 MIDI OUT, J3 MIDI IN, M1 Mounting, M2 Mounting, M3 Mounting, M4 Mounting, U1 6N138, U2 LM7805_TO220, U3 74LS00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

Commit message: Reordered IDC pins
Parts:
- J1: footprint Connector_IDC:IDC-Header_2x13_P2.54mm_Vertical -> DB25_Serial:DB25_Serial_IDC
Changed lines of the file:
@@
 F 0 "J1" H 3525 3392 50  0000 C CNN
 F 1 "Amiga Serial" H 3525 3301 50  0000 C CNN
-F 2 "Connector_IDC:IDC-Header_2x13_P2.54mm_Vertical" H 3475 2575 50  0001 C CNN
+F 2 "DB25_Serial:DB25_Serial_IDC" H 3475 2575 50  0001 C CNN
 F 3 "~" H 3475 2575 50  0001 C CNN
 	1    3475 2575

Commit message: Specify correct MAX232A variant
Parts:
- U4: value MAX232 -> MAX232A
Changed lines of the file:
@@
 P 2850 5875
 F 0 "U4" H 2850 6325 50  0000 C CNN
-F 1 "MAX232" H 2850 6225 50  0000 C CNN
+F 1 "MAX232A" H 2850 6225 50  0000 C CNN
 F 2 "Package_DIP:DIP-16_W7.62mm_Socket_LongPads" H 2900 4825 50  0001 L CNN
 F 3 "http://www.ti.com/lit/ds/symlink/max232.pdf" H 2850 5975 50  0001 C CNN
