File: BulkyMIDI-32 Channel Panel/BulkyMIDI-32 Channel Panel.kicad_pcb (KiCad board)
At the start: 2 copper layers, 100 x 23.2 mm, 22 parts, among them J1 Channel_Panel, M1 Mounting_Pin, M2 Mounting_Pin, M3 Mounting_Pin, M4 Mounting_Pin

Commit message: Added VU SIDi front panel
Other:
- board text added: "BulkyMIDI-32 Channel Panel (rev. A) github.com/tebl"
