File: BulkyMIDI-32 Play Panel/BulkyMIDI-32 Play Panel.sch (KiCad schematic (older format))
At the start: 11 parts, among them IC1 0.91_I2C_OLED, J1 Play_Panel, M1 Mounting_Pin, M2 Mounting_Pin, M3 Mounting_Pin, M4 Mounting_Pin

Commit message: Added Play FP1 and a post for holding OLED
Parts:
- added M5: Mounting_Pin, mounting:M3_pin, symbol mounting:Mounting_Pin
Connections:
- net GND: now also M5.1
Changed lines of the file:
@@
 L mounting:Mounting_Pin M1
 U 1 1 6282631C
+P 10600 575
+F 0 "M1" H 10600 675 50  0001 C CNN
+F 1 "Mounting_Pin" H 10600 500 50  0001 C CNN
+F 2 "mounting:M3_pin" H 10600 575 50  0001 C CNN
+F 3 "~" H 10600 575 50  0001 C CNN
+	1    10600 575
+	1    0    0    -1
+$EndComp
+$Comp
+L mounting:Mounting_Pin M2
+U 1 1 62826824
 P 10725 575
-F 0 "M1" H 10725 675 50  0001 C CNN
+F 0 "M2" H 10725 675 50  0001 C CNN
 F 1 "Mounting_Pin" H 10725 500 50  0001 C CNN
 F 2 "mounting:M3_pin" H 10725 575 50  0001 C CNN
@@
 $EndComp
 $Comp
-L mounting:Mounting_Pin M2
-U 1 1 62826824
+L mounting:Mounting_Pin M3
+U 1 1 62826D8F
 P 10850 575
-F 0 "M2" H 10850 675 50  0001 C CNN
+F 0 "M3" H 10850 675 50  0001 C CNN
 F 1 "Mounting_Pin" H 10850 500 50  0001 C CNN
 F 2 "mounting:M3_pin" H 10850 575 50  0001 C CNN
@@
 $EndComp
 $Comp
-L mounting:Mounting_Pin M3
-U 1 1 62826D8F
+L mounting:Mounting_Pin M4
+U 1 1 62827110
 P 10975 575
-F 0 "M3" H 10975 675 50  0001 C CNN
+F 0 "M4" H 10975 675 50  0001 C CNN
 F 1 "Mounting_Pin" H 10975 500 50  0001 C CNN
 F 2 "mounting:M3_pin" H 10975 575 50  0001 C CNN
 F 3 "~" H 10975 575 50  0001 C CNN
 	1    10975 575
-	1    0    0    -1
-$EndComp
-$Comp
-L mounting:Mounting_Pin M4
-U 1 1 62827110
-P 11100 575
-F 0 "M4" H 11100 675 50  0001 C CNN
-F 1 "Mounting_Pin" H 11100 500 50  0001 C CNN
-F 2 "mounting:M3_pin" H 11100 575 50  0001 C CNN
-F 3 "~" H 11100 575 50  0001 C CNN
-	1    11100 575
 	1    0    0    -1
 $EndComp
@@
 $EndComp
 Wire Wire Line
+	10600 725  10600 800
+Wire Wire Line
+	10600 800  10725 800
+Wire Wire Line
+	10975 800  10975 725
+Wire Wire Line
 	10725 725  10725 800
+Connection ~ 10725 800
 Wire Wire Line
 	10725 800  10850 800
-Wire Wire Line
-	11100 800  11100 725
 Wire Wire Line
 	10850 725  10850 800
@@
 	10850 800  10975 800
 Wire Wire Line
-	10975 725  10975 800
-Connection ~ 10975 800
-Wire Wire Line
-	10975 800  11100 800
-Wire Wire Line
 	11100 800  11100 875
-Connection ~ 11100 800
 Wire Wire Line
 	4975 2600 4475 2600
@@
 NoConn ~ 4475 3800
 NoConn ~ 4475 3900
+$Comp
+L mounting:Mounting_Pin M5
+U 1 1 6292635F
+P 11100 575
+F 0 "M5" H 11100 675 50  0001 C CNN
+F 1 "Mounting_Pin" H 11100 500 50  0001 C CNN
+F 2 "mounting:M3_pin" H 11100 575 50  0001 C CNN
+F 3 "~" H 11100 575 50  0001 C CNN
+	1    11100 575
+	1    0    0    -1
+$EndComp
+Wire Wire Line
+	10975 800  11100 800
+Connection ~ 10975 800
+Wire Wire Line
+	11100 800  11100 725
+Connection ~ 11100 800
 Wire Bus Line
 	5275 5150 5275 5600

Commit message: Schematic tweak
Changed lines of the file:
@@
 L power:GND #PWR0111
 U 1 1 6282AADA
-P 11100 875
-F 0 "#PWR0111" H 11100 625 50  0001 C CNN
-F 1 "GND" H 11105 702 50  0000 C CNN
-F 2 "" H 11100 875 50  0001 C CNN
-F 3 "" H 11100 875 50  0001 C CNN
-	1    11100 875
+P 10975 875
+F 0 "#PWR0111" H 10975 625 50  0001 C CNN
+F 1 "GND" H 10980 702 50  0000 C CNN
+F 2 "" H 10975 875 50  0001 C CNN
+F 3 "" H 10975 875 50  0001 C CNN
+	1    10975 875
 	1    0    0    -1
 $EndComp
@@
 	10850 800  10975 800
 Wire Wire Line
-	11100 800  11100 875
+	10975 800  10975 875
 Wire Wire Line
 	4975 2600 4475 2600
@@
 L mounting:Mounting_Pin M5
 U 1 1 6292635F
-P 11100 575
-F 0 "M5" H 11100 675 50  0001 C CNN
-F 1 "Mounting_Pin" H 11100 500 50  0001 C CNN
-F 2 "mounting:M3_pin" H 11100 575 50  0001 C CNN
-F 3 "~" H 11100 575 50  0001 C CNN
-	1    11100 575
-	1    0    0    -1
-$EndComp
-Wire Wire Line
-	10975 800  11100 800
+P 7090 2450
+F 0 "M5" H 7090 2550 50  0001 C CNN
+F 1 "Mounting_Pin" H 7090 2375 50  0001 C CNN
+F 2 "mounting:M3_pin" H 7090 2450 50  0001 C CNN
+F 3 "~" H 7090 2450 50  0001 C CNN
+	1    7090 2450
+	1    0    0    -1
+$EndComp
 Connection ~ 10975 800
-Wire Wire Line
-	11100 800  11100 725
-Connection ~ 11100 800
+$Comp
+L power:GND #PWR?
+U 1 1 62937337
+P 7090 2700
+F 0 "#PWR?" H 7090 2450 50  0001 C CNN
+F 1 "GND" H 7095 2527 50  0000 C CNN
+F 2 "" H 7090 2700 50  0001 C CNN
+F 3 "" H 7090 2700 50  0001 C CNN
+	1    7090 2700
+	1    0    0    -1
+$EndComp
+Wire Wire Line
+	7090 2700 7090 2600
 Wire Bus Line
 	5275 5150 5275 5600
