File: BulkyMIDI-32 Channel 2/BulkyMIDI-32 Channel 2.kicad_pcb (KiCad board)
At the start: 2 copper layers, 100 x 100 mm, 103 parts, among them J1 DC IN, J2 MIDI THRU, J3 MIDI IN, J4 Panel, J5 Conn_Power, J6 MODE, J7 TRS_3.5mm, J8 Breakout, M1 Mounting, M2 Mounting, M3 Mounting, M4 Mounting, Q10 2N3904, Q11 2N3904, Q12 2N3904, Q13 2N3904, Q14 2N3904, Q15 2N3904, Q16 2N3904, Q17 2N3904, Q2 2N3904, Q3 2N3904, Q4 2N3904, Q5 2N3904, Q6 2N3904, Q7 2N3904, Q8 2N3904, Q9 2N3904, SW1 SELECT, U1 74HCT14, U2 74HC595, U3 6N138, U4 74HC595

Commit message: Build tweaks
Parts:
- U1: footprint Package_DIP:DIP-14_W7.62mm -> Package_DIP:DIP-14_W7.62mm_Socket_LongPads
- moved C3 1.27 mm to (86.9, 101.8), turned to 180 degrees
- moved C5 1.27 mm to (86.9, 111.8), turned to 180 degrees
Connections:
- C3 pad 1: Net-(C3-Pad1) -> VU_R
- C3 pad 2: VU_R -> Net-(C3-Pad2)
- C5 pad 1: Net-(C5-Pad1) -> VU_L
- C5 pad 2: VU_L -> Net-(C5-Pad2)
- J7 pad 2: Net-(C3-Pad1) -> Net-(C3-Pad2)
- J7 pad 5: Net-(C5-Pad1) -> Net-(C5-Pad2)
Routing:
- net Net-(C5-Pad1): track 6.65 -> 0.00 mm
- net Net-(C3-Pad1): track 6.65 -> 0.00 mm
- net Net-(C5-Pad2): track 0.00 -> 5.92 mm
- net Net-(C3-Pad2): track 0.00 -> 5.92 mm
- net Net-(U1-Pad10): track 13.2 -> 15.1 mm
- net MIDI_IN: track 71.8 -> 73.1 mm
- net VU_L: track 72.6 -> 73.3 mm
Other:
- board text added: "BulkyMIDI-32 Channel 2 (rev. B) github.com/tebl"
- board text removed: "BulkyMIDI-32 Channel 2 (rev. A) github.com/tebl"
