File: BulkyMIDI-32 Channel 2/BulkyMIDI-32 Channel 2.sch (KiCad schematic (older format))
At the start: 102 parts, among them J1 DC IN, J2 MIDI THRU, J3 MIDI IN, J4 Panel, J5 Conn_Power, J6 MODE, J7 TRS_3.5mm, J8 Breakout, M1 Mounting, M2 Mounting, M3 Mounting, M4 Mounting, Q10 2N3904, Q11 2N3904, Q12 2N3904, Q13 2N3904, Q14 2N3904, Q15 2N3904, Q16 2N3904, Q17 2N3904, Q2 2N3904, Q3 2N3904, Q4 2N3904, Q5 2N3904, Q6 2N3904, Q7 2N3904, Q8 2N3904, Q9 2N3904, SW1 SELECT, U1 74HCT14, U2 74HC595, U3 6N138, U4 74HC595

Commit message: Build tweaks
Parts:
- U1: footprint Package_DIP:DIP-14_W7.62mm -> Package_DIP:DIP-14_W7.62mm_Socket_LongPads
Connections:
- net VU_L: now also C5.1; no longer C5.2
- net VU_R: now also C3.1; no longer C3.2
- net at J7.2: now also C3.2; no longer C3.1
- net at J7.5: now also C5.2; no longer C5.1
Changed lines of the file:
@@
 F 0 "U1" H 4675 3625 50  0000 C CNN
 F 1 "74HCT14" H 4675 3550 50  0000 C CNN
-F 2 "Package_DIP:DIP-14_W7.62mm" H 4675 3350 50  0001 C CNN
+F 2 "Package_DIP:DIP-14_W7.62mm_Socket_LongPads" H 4675 3350 50  0001 C CNN
 F 3 "http://www.ti.com/lit/gpn/sn74HC14" H 4675 3350 50  0001 C CNN
 	4    4675 3350
@@
 F 0 "U1" H 4775 2175 50  0000 C CNN
 F 1 "74HCT14" H 4775 2100 50  0000 C CNN
-F 2 "Package_DIP:DIP-14_W7.62mm" H 4775 2350 50  0001 C CNN
+F 2 "Package_DIP:DIP-14_W7.62mm_Socket_LongPads" H 4775 2350 50  0001 C CNN
 F 3 "http://www.ti.com/lit/gpn/sn74HC14" H 4775 2350 50  0001 C CNN
 	5    4775 2350
@@
 F 0 "U1" H 5525 2175 50  0000 C CNN
 F 1 "74HCT14" H 5525 2100 50  0000 C CNN
-F 2 "Package_DIP:DIP-14_W7.62mm" H 5525 2350 50  0001 C CNN
+F 2 "Package_DIP:DIP-14_W7.62mm_Socket_LongPads" H 5525 2350 50  0001 C CNN
 F 3 "http://www.ti.com/lit/gpn/sn74HC14" H 5525 2350 50  0001 C CNN
 	6    5525 2350
@@
 F 0 "U1" V 11083 10275 50  0000 C CNN
 F 1 "74HCT14" V 11174 10275 50  0000 C CNN
-F 2 "Package_DIP:DIP-14_W7.62mm" H 11450 10275 50  0001 C CNN
+F 2 "Package_DIP:DIP-14_W7.62mm_Socket_LongPads" H 11450 10275 50  0001 C CNN
 F 3 "http://www.ti.com/lit/gpn/sn74HC14" H 11450 10275 50  0001 C CNN
 	7    11450 10275
@@
 F 0 "U1" H 5400 4275 50  0000 C CNN
 F 1 "74HCT14" H 5400 4200 50  0000 C CNN
-F 2 "Package_DIP:DIP-14_W7.62mm" H 5400 4000 50  0001 C CNN
+F 2 "Package_DIP:DIP-14_W7.62mm_Socket_LongPads" H 5400 4000 50  0001 C CNN
 F 3 "http://www.ti.com/lit/gpn/sn74HC14" H 5400 4000 50  0001 C CNN
 	1    5400 4000
@@
 F 0 "U1" H 4675 4275 50  0000 C CNN
 F 1 "74HCT14" H 4675 4200 50  0000 C CNN
-F 2 "Package_DIP:DIP-14_W7.62mm" H 4675 4000 50  0001 C CNN
+F 2 "Package_DIP:DIP-14_W7.62mm_Socket_LongPads" H 4675 4000 50  0001 C CNN
 F 3 "http://www.ti.com/lit/gpn/sn74HC14" H 4675 4000 50  0001 C CNN
 	2    4675 4000
@@
 F 0 "U1" H 9300 10675 50  0000 C CNN
 F 1 "74HCT14" H 9300 10600 50  0000 C CNN
-F 2 "Package_DIP:DIP-14_W7.62mm" H 9300 10400 50  0001 C CNN
+F 2 "Package_DIP:DIP-14_W7.62mm_Socket_LongPads" H 9300 10400 50  0001 C CNN
 F 3 "http://www.ti.com/lit/gpn/sn74HC14" H 9300 10400 50  0001 C CNN
 	3    9300 10400
@@
 U 1 1 65188134
 P 2175 5625
-F 0 "C3" V 1950 5625 50  0000 C CNN
-F 1 "10uF" V 2041 5625 50  0000 C CNN
+F 0 "C3" V 2350 5625 50  0000 C CNN
+F 1 "10uF" V 2275 5625 50  0000 C CNN
 F 2 "Capacitor_THT:CP_Radial_D4.0mm_P2.00mm" H 2175 5625 50  0001 C CNN
 F 3 "~" H 2175 5625 50  0001 C CNN
 	1    2175 5625
-	0    -1   1    0
+	0    1    -1   0
 $EndComp
 $Comp
@@
 U 1 1 6518D765
 P 2175 5875
-F 0 "C5" V 2050 5875 50  0000 C CNN
-F 1 "10uF" V 1975 5875 50  0000 C CNN
+F 0 "C5" V 2275 5875 50  0000 C CNN
+F 1 "10uF" V 2350 5875 50  0000 C CNN
 F 2 "Capacitor_THT:CP_Radial_D4.0mm_P2.00mm" H 2175 5875 50  0001 C CNN
 F 3 "~" H 2175 5875 50  0001 C CNN
 	1    2175 5875
-	0    -1   -1   0
-$EndComp
-Wire Wire Line
+	0    1    1    0
+$EndComp
+Wire Wire Line
