File: BulkyMIDI-32 Channel/BulkyMIDI-32 Channel.kicad_pcb (KiCad board)
At the start: 2 copper layers, 100 x 100 mm, 122 parts, among them J1 DC IN, J2 MIDI THRU, J3 MIDI IN, J4 Panel, J5 Conn_Power, M1 Mounting, M2 Mounting, M3 Mounting, M4 Mounting, Q1 2N3906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

Commit message: Silkscreen tweaks
Other:
- board text added: "MIDI IN"
- board text added: "MIDI THRU"
- board text removed: "MIDI IN (MCU)"
- board text removed: "MIDI OUT (MCU)"

Commit message: Wrong capacitor value
Parts:
- C10, C27: value 68nF -> 68pF
