File: BulkyMIDI-32 Module Panel/BulkyMIDI-32 Module Panel.kicad_pcb (KiCad board)
At the start: 2 copper layers, 100 x 23.2 mm, 14 parts, among them IC1 OLED, J1 Module Panel, M1 Mounting_Pin, M2 Mounting_Pin, M3 Mounting_Pin, M4 Mounting_Pin, SW1 SYNTH, SW2 ROM

Commit message: Module FP1 sketched out
Parts:
- moved SW2 7.64 mm to (117.3, 121.6), turned to 90 degrees
- moved SW1 4.85 mm to (108.6, 121.6), turned to 90 degrees
Routing:
- net /ROM: track 74.3 -> 54.4 mm
- net /SYNTH: track 51.6 -> 69.5 mm
- net /PWR: track 67.8 -> 70.5 mm
