File: BulkyMIDI-32 Audio Switch/Channels.sch (KiCad schematic (older format))
At the start: 48 parts, among them J2 CH2, J3 CH1, J5 CH3, J7 CH4, J8 CH5, J9 CH6, K1 HK19F-DC, K2 HK19F-DC, K3 HK19F-DC, K4 HK19F-DC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

Commit message: Untested audio switch module
Parts:
- removed D13: CH4, LED_THT:LED_D3.0mm, symbol Device:LED
- removed D14: CH5, LED_THT:LED_D3.0mm, symbol Device:LED
- removed D15: CH6, LED_THT:LED_D3.0mm, symbol Device:LED
- removed D7: CH2, LED_THT:LED_D3.0mm, symbol Device:LED
- removed D8: CH1, LED_THT:LED_D3.0mm, symbol Device:LED
- removed D9: CH3, LED_THT:LED_D3.0mm, symbol Device:LED
- Q1, Q2, Q3, Q4, Q5, Q6: footprint Package_TO_SOT_THT:TO-92_Inline -> Package_TO_SOT_THT:TO-92_Inline_Wide
- R10, R11, R12, R13, R14, R15, R16, R17, R18, R19, R20, R21, R22, R23, R24, R25, R26, R27: footprint Resistor_THT:R_Axial_DIN0207_L6.3mm_D2.5mm_P10.16mm_Horizontal -> resistor:R_Axial_DIN0207_L6.3mm_D2.5mm_P10.16mm_Horizontal
- renumbered K2 to K1, K1 to K2

Commit message: Fix weird socket selection
Changed lines of the file:
@@
 	-1   0    0    -1
 $EndComp
-Text HLabel 1150 2175 0    50   Input ~ 0
-CH1
-Text HLabel 1150 1450 0    50   Input ~ 0
+Text HLabel 1150 1450 0    50   Output ~ 0
 LED1
 $Comp
@@
 Text HLabel 5725 2175 0    50   Input ~ 0
 CH4
-Text HLabel 5725 1450 0    50   Input ~ 0
+Text HLabel 5725 1450 0    50   Output ~ 0
 LED4
 $Comp
@@
 Text HLabel 1150 4300 0    50   Input ~ 0
 CH2
-Text HLabel 1150 3575 0    50   Input ~ 0
+Text HLabel 1150 3575 0    50   Output ~ 0
 LED2
 $Comp
@@
 Text HLabel 5725 4300 0    50   Input ~ 0
 CH5
-Text HLabel 5725 3575 0    50   Input ~ 0
+Text HLabel 5725 3575 0    50   Output ~ 0
 LED5
 $Comp
@@
 Text HLabel 1150 6400 0    50   Input ~ 0
 CH3
-Text HLabel 1150 5675 0    50   Input ~ 0
+Text HLabel 1150 5675 0    50   Output ~ 0
 LED3
 $Comp
@@
 Text HLabel 5725 6400 0    50   Input ~ 0
 CH6
-Text HLabel 5725 5675 0    50   Input ~ 0
+Text HLabel 5725 5675 0    50   Output ~ 0
 LED6
 $Comp
@@
 Wire Wire Line
 	9575 1500 9500 1500
+Text HLabel 1150 2175 0    50   Input ~ 0
+CH1
 $EndSCHEMATC
