File: BulkyMIDI-32 Audio Switch Panel/BulkyMIDI-32 Audio Switch Panel.kicad_pcb (KiCad board)
At the start: 2 copper layers, 100 x 23.2 mm, 18 parts, among them J1 Switch Panel, M1 Mounting_Pin, M2 Mounting_Pin, M3 Mounting_Pin, M4 Mounting_Pin, SW1 CH1, SW2 CH2, SW3 CH3, SW4 CH4, SW5 CH5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

Commit message: Audio Switch FP1
Other:
- board text added: "JLCJLCJLCJLC"
