File: BulkyMIDI-32 Play/BulkyMIDI-32 Play.kicad_pcb (KiCad board)
At the start: 2 copper layers, 100 x 100 mm, 46 parts, among them IC1 0.91_I2C_OLED, J1 DC IN, J10 MIDI IN (ALT), J11 MIDI OUT (ALT), J2 MIDI OUT, J3 MIDI IN, J4 Conn_Power, J5 MIDI THRU, J6 Play_Panel, M1 Mounting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

Commit message: Build tweaks
Parts:
- U1: footprint Package_DIP:DIP-14_W7.62mm -> Package_DIP:DIP-14_W7.62mm_Socket_LongPads
Routing:
- net Net-(U1-Pad10): track 13.2 -> 15.1 mm
Other:
- board text added: "BulkyMIDI-32 Play (rev. B) github.com/tebl"
- board text removed: "BulkyMIDI-32 Play (rev. A) github.com/tebl"

Commit message: Forgotten gate
Connections:
- U1 pad 5: (no net) -> GND

Commit message: Modules worked more reliably when run through the onboard regulator
Parts:
- moved C6 35.6 mm to (106.7, 98.4), turned to 90 degrees
Connections:
- A1 pad 24: (no net) -> VIN
- J1 pad 1: +5V -> VIN
- J4 pad 1: +5V -> VIN
Routing:
- net +5V: track 519.0 -> 420.2 mm, vias 5 -> 6
- net VIN: track 0.00 -> 55.2 mm
- net MIDI_OUT: track 76.4 -> 73.9 mm
- net MIDI_IN: track 73.9 -> 71.4 mm
Other:
- rule trace_min: 0.2 -> 0
