File: adapters/MIDI Breakout Board/MIDI Breakout Board.sch (KiCad schematic (older format))
At the start: 14 parts, among them J1 MIDI, J2 MIDI OUT, J3 MIDI IN, M1 Mounting_Pin, M2 Mounting_Pin, U1 6N138, U3 74LS00

Commit message: Add pulldown to breakout board
Parts:
- added R5: 4k7, Resistor_THT:R_Axial_DIN0207_L6.3mm_D2.5mm_P10.16mm_Horizontal, symbol Device:R
Connections:
- net GND: now also R5.1
- net at U1.7 (VO1): now also R5.2
- no-connect marks 6 -> 5
Changed lines of the file:
@@
 Title "MIDI Breakout Board"
 Date ""
-Rev "A"
+Rev "B"
 Comp ""
 Comment1 ""
@@
 Wire Wire Line
 	5600 1950 5525 1950
-NoConn ~ 7450 1950
 $Comp
 L power:+5V #PWR0104
@@
 L power:GND #PWR0105
 U 1 1 6212BC17
-P 7525 2350
-F 0 "#PWR0105" H 7525 2100 50  0001 C CNN
-F 1 "GND" H 7530 2177 50  0000 C CNN
-F 2 "" H 7525 2350 50  0001 C CNN
-F 3 "" H 7525 2350 50  0001 C CNN
-	1    7525 2350
-	1    0    0    -1
-$EndComp
-Wire Wire Line
-	7525 2250 7525 2350
+P 7525 2775
+F 0 "#PWR0105" H 7525 2525 50  0001 C CNN
+F 1 "GND" H 7530 2602 50  0000 C CNN
+F 2 "" H 7525 2775 50  0001 C CNN
+F 3 "" H 7525 2775 50  0001 C CNN
+	1    7525 2775
+	1    0    0    -1
+$EndComp
 Wire Wire Line
 	7450 2250 7525 2250
@@
 	11125 775  11125 850
 Connection ~ 11125 775
+$Comp
+L Device:R R5
+U 1 1 62F00614
+P 7600 2475
+F 0 "R5" H 7525 2525 50  0000 R CNN
+F 1 "4k7" H 7550 2450 50  0000 R CNN
+F 2 "Resistor_THT:R_Axial_DIN0207_L6.3mm_D2.5mm_P10.16mm_Horizontal" V 7530 2475 50  0001 C CNN
+F 3 "~" H 7600 2475 50  0001 C CNN
+	1    7600 2475
+	-1   0    0    1
+$EndComp
+Wire Wire Line
+	7525 2250 7525 2700
+Wire Wire Line
+	7600 2625 7600 2700
+Wire Wire Line
+	7600 2700 7525 2700
+Connection ~ 7525 2700
+Wire Wire Line
+	7525 2700 7525 2775
+Wire Wire Line
+	7600 2325 7600 1950
+Wire Wire Line
+	7600 1950 7450 1950
 $EndSCHEMATC
