File: BulkyMIDI-32 Input Switch/BulkyMIDI-32 Input Switch.kicad_pcb (KiCad board)
At the start: 2 copper layers, 100 x 100 mm, 86 parts, among them J1 DC IN, J2 MIDI IN4, J2 MIDI THRU, J3 MIDI IN1, J3 MIDI IN2, J4 Conn_Power, J5 MIDI IN3, J6 Switch Panel, K1 HK19F-DC, K2 HK19F-DC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

Commit message: Initial layout done
Parts:
- removed the C9 at (31.5, 115.6)
- removed D17, D18, D6: 1N4148, Diode_THT:D_DO-35_SOD27_P7.62mm_Horizontal
- removed the J2 at (157.5, 125.1)
- removed the J2 at (147.2, 141.9)
- removed the J2 at (157.5, 104.8)
- removed the J2 at (153.0, 67.3)
- removed the J3 at (132.7, 67.3)
- removed K5, K6: HK19F-DC, HK19F-DC:HK19F-DC
- removed Q5, Q6: 2N3904, Package_TO_SOT_THT:TO-92_Inline_Wide
- added C3: 100nF, Capacitor_THT:C_Disc_D4.7mm_W2.5mm_P5.00mm, F.Cu at (96.5, 71.1)
- added J10: MIDI THRU3, BulkyMIDI-32:DIN5_MIDI, F.Cu at (157.5, 125.1)
- added J2: MIDI IN1, BulkyMIDI-32:DIN5_MIDI, F.Cu at (132.7, 67.3)
- added J7: MIDI IN4, BulkyMIDI-32:DIN5_MIDI, F.Cu at (152.7, 141.9)
- added J8: MIDI THRU1, BulkyMIDI-32:DIN5_MIDI, F.Cu at (153.0, 67.3)
- added J9: MIDI THRU2, BulkyMIDI-32:DIN5_MIDI, F.Cu at (157.5, 104.8)
- added R29: 4k7, Resistor_THT:R_Axial_DIN0207_L6.3mm_D2.5mm_P10.16mm_Horizontal, F.Cu at (97.2, 96.5)
- added U2: 6N138, Package_DIP:DIP-8_W7.62mm_Socket_LongPads, F.Cu at (81.9, 98.4)
- added U3: 74HCT14, Package_DIP:DIP-14_W7.62mm_Socket_LongPads, F.Cu at (90.2, 74.9)
- J6: value Switch Panel -> Input Panel; footprint BulkyMIDI-32:Switch_Panel -> BulkyMIDI-32:Input_Panel
- R20, R21: value 1k -> 220; footprint resistor:R_Axial_DIN0207_L6.3mm_D2.5mm_P10.16mm_Horizontal -> Resistor_THT:R_Axial_DIN0207_L6.3mm_D2.5mm_P10.16mm_Horizontal
- R23, R24: value 10k -> 220; footprint resistor:R_Axial_DIN0207_L6.3mm_D2.5mm_P10.16mm_Horizontal -> Resistor_THT:R_Axial_DIN0207_L6.3mm_D2.5mm_P10.16mm_Horizontal
- R26, R27: value 470 -> 220; footprint resistor:R_Axial_DIN0207_L6.3mm_D2.5mm_P10.16mm_Horizontal -> Resistor_THT:R_Axial_DIN0207_L6.3mm_D2.5mm_P10.16mm_Horizontal
- R5: value 100k -> 220; footprint resistor:R_Axial_DIN0207_L6.3mm_D2.5mm_P10.16mm_Horizontal -> Resistor_THT:R_Axial_DIN0207_L6.3mm_D2.5mm_P10.16mm_Horizontal
- R6: value 100k -> 2k2; footprint resistor:R_Axial_DIN0207_L6.3mm_D2.5mm_P10.16mm_Horizontal -> Resistor_THT:R_Axial_DIN0207_L6.3mm_D2.5mm_P10.16mm_Horizontal
- moved R26 171.5 mm to (167.6, 62.2), turned to 270 degrees
- moved K4 162.5 mm to (130.8, 123.8), turned to 0 degrees
- moved Q4 152.6 mm to (129.3, 132.7)
- moved R19 152.6 mm to (133.1, 128.3)
- moved R22 152.6 mm to (143.3, 132.1)
- moved K3 148.4 mm to (131.1, 103.9), turned to 0 degrees
- moved K1 147.2 mm to (131.1, 84.2), turned to 0 degrees
- moved D16 144.7 mm to (127.6, 123.8), turned to 90 degrees
- moved D12 142.2 mm to (127.9, 103.9), turned to 90 degrees
- moved D11 140.9 mm to (127.9, 84.2), turned to 90 degrees
- moved G*** 139.5 mm to (76.8, 125.7), turned to 90 degrees
- moved R24 138.7 mm to (164.5, 62.2), turned to 270 degrees
- moved Q2 133.1 mm to (129.3, 92.7)
- moved R11 133.1 mm to (133.1, 88.3)
- moved R14 133.1 mm to (143.3, 92.1)
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- renumbered C3 to C9
Connections:
- C8 pad 1: /SW5 -> GND
- C8 pad 2: GND -> +5V
- D5 pad 1: Net-(D1-Pad1) -> Net-(D5-Pad1)
- D5 pad 2: /SW5 -> MIDI_P5
- J3 pad 4: (no net) -> Net-(J3-Pad4)
- J3 pad 5: (no net) -> Net-(J3-Pad5)
- J5 pad 4: (no net) -> Net-(J5-Pad4)
- J5 pad 5: (no net) -> Net-(J5-Pad5)
- J6 pad 12: /SW5 -> (no net)
- J6 pad 13: /LED5 -> (no net)
- J6 pad 14: /SW6 -> GND
- J6 pad 15: /LED6 -> +5V
- K1 pad 13: /LEFT -> MIDI_P4
- K1 pad 4: /RIGHT -> MIDI_P5
- K2 pad 13: /LEFT -> MIDI_P4
- K2 pad 4: /RIGHT -> MIDI_P5
- K2 pad 8: Net-(J2-Pad2) -> Net-(J3-Pad5)
- K2 pad 9: Net-(J2-Pad5) (its old number) -> Net-(J3-Pad4)
- K3 pad 13: /LEFT -> MIDI_P4
- K3 pad 4: /RIGHT -> MIDI_P5
- K3 pad 8: Net-(J5-Pad2) -> Net-(J5-Pad5)
- K3 pad 9: Net-(J5-Pad5) -> Net-(J5-Pad4)
- K4 pad 13: /LEFT -> MIDI_P4
- K4 pad 4: /RIGHT -> MIDI_P5
- R20 pad 1: Net-(Q5-Pad2) -> Net-(J8-Pad5)
- R20 pad 2: /CH5 -> Net-(R20-Pad2)
- R21 pad 1: Net-(Q6-Pad2) -> Net-(J9-Pad5)
- R21 pad 2: /CH6 -> Net-(R21-Pad2)
- R23 pad 1: GND -> Net-(J10-Pad5)
- R23 pad 2: Net-(Q5-Pad2) -> Net-(R23-Pad2)
- R24 pad 1: GND -> +5V
- R24 pad 2: Net-(Q6-Pad2) -> Net-(J8-Pad4)
- R26 pad 1: Net-(D17-Pad2) -> +5V
- R26 pad 2: /LED5 -> Net-(J9-Pad4)
- R27 pad 1: Net-(D18-Pad2) -> +5V
- R27 pad 2: /LED6 -> Net-(J10-Pad4)
- R5 pad 1: /SW5 -> Net-(D5-Pad1)
- R5 pad 2: GND -> MIDI_P4
- R6 pad 1: /SW6 -> +5V
- R6 pad 2: GND -> Net-(R6-Pad2)
- U1 pad 12: /CH5 -> (no net)
- U1 pad 13: /SW5 -> GND
- U1 pad 14: /SW6 -> GND
- U1 pad 15: /CH6 -> (no net)
Routing:
- net +5V: track 326.6 -> 597.8 mm, vias 0 -> 1
- net MIDI_P4: track 0.00 -> 160.7 mm, vias 0 -> 3
- net MIDI_P5: track 0.00 -> 124.4 mm, vias 0 -> 2
- net Net-(J9-Pad5): track 0.00 -> 123.2 mm
- net /RIGHT: track 111.2 -> 0.00 mm
- net /LEFT: track 104.9 -> 0.00 mm
- net Net-(D18-Pad2): track 89.5 -> 0.00 mm
- net Net-(J10-Pad5): track 0.00 -> 77.3 mm, vias 0 -> 2
- net Net-(D17-Pad2): track 76.5 -> 0.00 mm
- net Net-(J8-Pad5): track 0.00 -> 73.5 mm
- net Net-(D12-Pad2): track 38.9 -> 110.0 mm, vias 1 -> 2
- net /CH5: track 69.6 -> 0.00 mm
- net /CH6: track 61.2 -> 0.00 mm
- net Net-(D16-Pad2): track 82.9 -> 30.9 mm
- net Net-(D10-Pad2): track 42.7 -> 94.5 mm
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Other:
- outline, holes or cut-outs redrawn
- board text added: "IN 1"
- board text added: "IN 2"
- board text added: "IN 3"
- board text added: "IN 4"
- board text added: "THRU 1"
- board text added: "THRU 2"
- board text added: "THRU 3"
- board text removed: "CH1"
- board text removed: "CH2"
- board text removed: "CH3"
- board text removed: "JLCJLCJLCJLC"
- board text removed: "OUTPUT"
