File: BulkyMIDI-32 Input Switch/BulkyMIDI-32 Input Switch.sch (KiCad schematic (older format))
At the start: 35 parts, among them J1 DC IN, J4 Conn_Power, J6 Input Panel, M1 Mounting, M2 Mounting, M3 Mounting, M4 Mounting, SW1 CH1, SW2 CH2, SW3 CH3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

Commit message: Initial layout done
Parts:
- J6: footprint BulkyMIDI-32:Switch_Panel -> BulkyMIDI-32:Input_Panel
Connections:
- net +5V: now also J6.15 (VCC)
- net GND: now also J6.14 (GND)
Changed lines of the file:
@@
 Entry Wire Line
 	10000 2600 9900 2500
-Wire Wire Line
-	10425 2500 10425 4300
 Connection ~ 10350 2400
 Wire Wire Line
@@
 	-1   0    0    -1
 $EndComp
-Connection ~ 10425 4300
-Wire Wire Line
-	10425 4450 10425 4300
 $Comp
 L power:GND #PWR0118
 U 1 1 635034D3
-P 10425 4450
-F 0 "#PWR0118" H 10425 4200 50  0001 C CNN
-F 1 "GND" H 10430 4277 50  0000 C CNN
-F 2 "" H 10425 4450 50  0001 C CNN
-F 3 "" H 10425 4450 50  0001 C CNN
-	1    10425 4450
+P 10425 3975
+F 0 "#PWR0118" H 10425 3725 50  0001 C CNN
+F 1 "GND" H 10430 3802 50  0000 C CNN
+F 2 "" H 10425 3975 50  0001 C CNN
+F 3 "" H 10425 3975 50  0001 C CNN
+	1    10425 3975
 	1    0    0    -1
 $EndComp
 Wire Wire Line
 	10350 2400 10500 2400
-Wire Wire Line
-	10350 4400 10350 2400
-Wire Wire Line
-	10500 4400 10350 4400
-Wire Wire Line
-	10425 4300 10500 4300
 Wire Wire Line
 	10500 2500 10425 2500
@@
 F 0 "J6" H 10718 4625 50  0000 C CNN
 F 1 "Input Panel" H 10718 4534 50  0000 C CNN
-F 2 "BulkyMIDI-32:Switch_Panel" H 10700 3400 50  0001 C CNN
+F 2 "BulkyMIDI-32:Input_Panel" H 10700 3400 50  0001 C CNN
 F 3 "~" H 10700 3400 50  0001 C CNN
 	1    10700 3400
@@
 Wire Wire Line
 	900  2825 900  4050
+Wire Wire Line
+	10425 2500 10425 3700
+Wire Wire Line
+	10500 3700 10425 3700
+Connection ~ 10425 3700
+Wire Wire Line
+	10425 3700 10425 3975
+Wire Wire Line
+	10500 3800 10350 3800
+Wire Wire Line
+	10350 3800 10350 2400
 Wire Bus Line
 	7925 2425 7925 2725
