File: BulkyMIDI-32 Input Switch/Channels.sch (KiCad schematic (older format))
At the start: 44 parts, among them J10 MIDI THRU3, J2 MIDI IN1, J3 MIDI IN2, J5 MIDI IN3, J7 MIDI IN4, J8 MIDI THRU1, J9 MIDI THRU2, K1 HK19F-DC, K2 HK19F-DC, K3 HK19F-DC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

Commit message: Initial layout done
Parts:
- added R29: 4k7, Resistor_THT:R_Axial_DIN0207_L6.3mm_D2.5mm_P10.16mm_Horizontal, symbol Device:R
Connections:
- net GND: now also R29.2
- net at U2.7 (VO1): now also R29.1
- no-connect marks 29 -> 28
Changed lines of the file:
@@
 	9275 1400 9350 1400
-$Comp
-L Isolator:6N138 U?
-U 1 1 63599E50
-P 6700 1300
-AR Path="/63599E50" Ref="U?"  Part="1"
-AR Path="/635D4EBA/63599E50" Ref="U2"  Part="1"
-F 0 "U2" H 6700 833 50  0000 C CNN
-F 1 "6N138" H 6700 924 50  0000 C CNN
-F 2 "Package_DIP:DIP-8_W7.62mm_Socket_LongPads" H 6990 1000 50  0001 C CNN
-F 3 "http://www.onsemi.com/pub/Collateral/HCPL2731-D.pdf" H 6990 1000 50  0001 C CNN
-	1    6700 1300
-	1    0    0    -1
-$EndComp
 $Comp
 L Device:R R?
@@
 	1    0    0    -1
 $EndComp
-NoConn ~ 7000 1200
 $Comp
 L power:+5V #PWR?
@@
 L power:GND #PWR?
 U 1 1 63599E9F
-P 7075 1600
+P 7175 1950
 AR Path="/63599E9F" Ref="#PWR?"  Part="1"
 AR Path="/635D4EBA/63599E9F" Ref="#PWR04"  Part="1"
-F 0 "#PWR04" H 7075 1350 50  0001 C CNN
-F 1 "GND" H 7080 1427 50  0000 C CNN
-F 2 "" H 7075 1600 50  0001 C CNN
-F 3 "" H 7075 1600 50  0001 C CNN
-	1    7075 1600
+F 0 "#PWR04" H 7175 1700 50  0001 C CNN
+F 1 "GND" H 7180 1777 50  0000 C CNN
+F 2 "" H 7175 1950 50  0001 C CNN
+F 3 "" H 7175 1950 50  0001 C CNN
+	1    7175 1950
 	1    0    0    -1
 $EndComp
@@
 Wire Wire Line
 	7000 1100 7075 1100
-Wire Wire Line
-	7075 1500 7075 1600
 Wire Wire Line
 	7000 1500 7075 1500
@@
 	10850 6225 10850 6300
 Connection ~ 10850 6225
+$Comp
+L Device:R R?
+U 1 1 63D9F837
+P 7175 1650
+AR Path="/63D9F837" Ref="R?"  Part="1"
+AR Path="/635D4EBA/63D9F837" Ref="R29"  Part="1"
+F 0 "R29" H 7100 1700 50  0000 R CNN
+F 1 "4k7" H 7125 1625 50  0000 R CNN
+F 2 "Resistor_THT:R_Axial_DIN0207_L6.3mm_D2.5mm_P10.16mm_Horizontal" V 7105 1650 50  0001 C CNN
+F 3 "~" H 7175 1650 50  0001 C CNN
+	1    7175 1650
+	-1   0    0    -1
+$EndComp
+$Comp
+L Isolator:6N138 U?
+U 1 1 63599E50
+P 6700 1300
+AR Path="/63599E50" Ref="U?"  Part="1"
+AR Path="/635D4EBA/63599E50" Ref="U2"  Part="1"
+F 0 "U2" H 6700 833 50  0000 C CNN
+F 1 "6N138" H 6700 924 50  0000 C CNN
+F 2 "Package_DIP:DIP-8_W7.62mm_Socket_LongPads" H 6990 1000 50  0001 C CNN
+F 3 "http://www.onsemi.com/pub/Collateral/HCPL2731-D.pdf" H 6990 1000 50  0001 C CNN
+	1    6700 1300
+	1    0    0    -1
+$EndComp
+Wire Wire Line
+	7000 1200 7175 1200
+Wire Wire Line
+	7175 1200 7175 1500
+Wire Wire Line
+	7175 1800 7175 1875
+Wire Wire Line
+	7175 1875 7075 1875
+Wire Wire Line
+	7075 1500 7075 1875
+Wire Wire Line
+	7175 1875 7175 1950
+Connection ~ 7175 1875
 $EndSCHEMATC
