File: BulkyMIDI-32 Dexed/BulkyMIDI-32 Dexed.kicad_pcb (KiCad board)
At the start: 2 copper layers, 100 x 100 mm, 44 parts, among them J1 DC IN, J2 MIDI OUT, J3 MIDI IN, J5 MIDI THRU, J7 Conn_Extras, J8 Dexed_Panel, M1 Mounting, M2 Mounting, M3 Mounting, M4 Mounting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

Commit message: Dexed changes
Parts:
- C10, C11, C12, C2, C7, C8, C9: value 10pF -> 10nF
- moved C12 4.02 mm to (144.8, 135.9)
- moved C11 3.42 mm to (141.6, 135.9)
- moved C10 2.84 mm to (138.4, 135.9)
- moved C9 2.29 mm to (135.3, 135.9)
- moved C8 1.80 mm to (132.1, 135.9)
- moved C7 1.42 mm to (128.9, 135.9)
- moved C2 1.27 mm to (125.7, 135.9)
Routing:
- net ENC_CLK: track 58.1 -> 60.4 mm
- net ENC_DAT: track 58.1 -> 59.9 mm
- net SW_DOWN: track 58.8 -> 60.1 mm
- net ENC_SW: track 53.9 -> 55.1 mm
- net +5V: track 279.6 -> 278.5 mm
- net SW_UP: track 60.6 -> 61.4 mm
- net Net-(R6-Pad1): track 40.9 -> 40.2 mm
Other:
- outline, holes or cut-outs redrawn
- board text added: "7x 10nF"
- board text added: "BulkyMIDI-32 Dexed (rev. B) github.com/tebl"
- board text removed: "7x 10pF"
- board text removed: "BulkyMIDI-32 Dexed (rev. A) github.com/tebl"
