File: BulkyMIDI-32 Dexed/BulkyMIDI-32 Dexed.sch (KiCad schematic (older format))
At the start: 38 parts, among them J1 DC IN, J2 MIDI OUT, J3 MIDI IN, J5 MIDI THRU, J7 Conn_Extras, J8 Dexed_Panel, M1 Mounting, M2 Mounting, M3 Mounting, M4 Mounting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

Commit message: Dexed changes
Parts:
- C10, C11, C12, C2, C7, C8, C9: value 10pF -> 10nF
Other:
- note added: "* The UP/DOWN buttons are strictly\nnot needed, they are included here\nin case someone who knows what\nthey're doing find a use for them."
Changed lines of the file:
@@
 P 11400 7925
 F 0 "C2" H 11425 8075 50  0000 L CNN
-F 1 "10pF" H 11425 8000 50  0000 L CNN
+F 1 "10nF" H 11425 8000 50  0000 L CNN
 F 2 "Capacitor_THT:C_Rect_L7.0mm_W2.0mm_P5.00mm" H 11438 7775 50  0001 C CNN
 F 3 "~" H 11400 7925 50  0001 C CNN
@@
 P 11675 7925
 F 0 "C7" H 11700 8075 50  0000 L CNN
-F 1 "10pF" H 11700 8000 50  0000 L CNN
+F 1 "10nF" H 11700 8000 50  0000 L CNN
 F 2 "Capacitor_THT:C_Rect_L7.0mm_W2.0mm_P5.00mm" H 11713 7775 50  0001 C CNN
 F 3 "~" H 11675 7925 50  0001 C CNN
@@
 P 11925 7925
 F 0 "C8" H 11950 8075 50  0000 L CNN
-F 1 "10pF" H 11950 8000 50  0000 L CNN
+F 1 "10nF" H 11950 8000 50  0000 L CNN
 F 2 "Capacitor_THT:C_Rect_L7.0mm_W2.0mm_P5.00mm" H 11963 7775 50  0001 C CNN
 F 3 "~" H 11925 7925 50  0001 C CNN
@@
 P 12175 7925
 F 0 "C9" H 12200 8075 50  0000 L CNN
-F 1 "10pF" H 12200 8000 50  0000 L CNN
+F 1 "10nF" H 12200 8000 50  0000 L CNN
 F 2 "Capacitor_THT:C_Rect_L7.0mm_W2.0mm_P5.00mm" H 12213 7775 50  0001 C CNN
 F 3 "~" H 12175 7925 50  0001 C CNN
@@
 P 12425 7925
 F 0 "C10" H 12450 8075 50  0000 L CNN
-F 1 "10pF" H 12450 8000 50  0000 L CNN
+F 1 "10nF" H 12450 8000 50  0000 L CNN
 F 2 "Capacitor_THT:C_Rect_L7.0mm_W2.0mm_P5.00mm" H 12463 7775 50  0001 C CNN
 F 3 "~" H 12425 7925 50  0001 C CNN
@@
 P 12675 7925
 F 0 "C11" H 12700 8075 50  0000 L CNN
-F 1 "10pF" H 12700 8000 50  0000 L CNN
+F 1 "10nF" H 12700 8000 50  0000 L CNN
 F 2 "Capacitor_THT:C_Rect_L7.0mm_W2.0mm_P5.00mm" H 12713 7775 50  0001 C CNN
 F 3 "~" H 12675 7925 50  0001 C CNN
@@
 P 12925 7925
 F 0 "C12" H 12950 8075 50  0000 L CNN
-F 1 "10pF" H 12950 8000 50  0000 L CNN
+F 1 "10nF" H 12950 8000 50  0000 L CNN
 F 2 "Capacitor_THT:C_Rect_L7.0mm_W2.0mm_P5.00mm" H 12963 7775 50  0001 C CNN
 F 3 "~" H 12925 7925 50  0001 C CNN
@@
 	12675 8100 12925 8100
 Connection ~ 12925 8100
+Text Notes 13625 7600 0    50   ~ 0
+* The UP/DOWN buttons are strictly\nnot needed, they are included here\nin case someone who knows what\nthey're doing find a use for them.
 $EndSCHEMATC
