File: BulkyMIDI-32 Internal Panel/BulkyMIDI-32 Internal Panel.kicad_pcb (KiCad board)
At the start: 2 copper layers, 100 x 22.5 mm, 19 parts, among them IC1 OLED, J1 Front Panel, M1 Mounting_Pin, M10 Mounting_Pad, M2 Mounting_Pin, M3 Mounting_Pin, M4 Mounting_Pin, M5 Mounting_Pad, M7 Mounting_Pad, M9 Mounting_Pad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

Commit message: Small changes to internal layout
Parts:
- moved IC1 0.50 mm to (134.3, 85.8)
Routing:
- net I2C_SDA: track 17.7 -> 18.7 mm
- net +3V3: track 29.9 -> 30.4 mm
Other:
- outline, holes or cut-outs redrawn
- board text added: "BulkyMIDI-32 Internal Panel (rev. B) github.com/tebl"
- board text removed: "BulkyMIDI-32 Internal Panel (rev. A) github.com/tebl"
