File: BulkyMIDI-32 ExModule/BulkyMIDI-32 ExModule.sch (KiCad schematic (older format))
At the start: 26 parts, among them J1 DC IN, J2 Wavetable, J3 MIDI IN, J4 AUDIO, J5 MIDI THRU, J6 ExModule_Panel, M1 Mounting, M2 Mounting, M3 Mounting, M4 Mounting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

Commit message: Add activity
Parts:
- added FB1: Wired Ferrite, Inductor_THT:L_Axial_L7.0mm_D3.3mm_P10.16mm_Horizontal_Fastron_MICC, symbol Device:Ferrite_Bead
Connections:
- net GND: now also FB1.2; no longer U1.1
- net GNDA: now also FB1.1
- net at U1.10, U1.13, U1.9: now also U1.1
- net Activity LED/MIDI: now reaches U1.2
- net Activity LED/Activity: now reaches R5.2
- no-connect marks 15 -> 14
Other:
- moved on the sheet: C6, C7, D1, D2, D3, D4, J1, J2, J3, J4, J5, J6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

Commit message: ExPower symbol
Parts:
- added A1: ExPower, symbol BulkyMIDI:ExModule_Power
Connections:
- net +12V: now also A1.3 (+12V)
- net +5V: now also A1.1 (5V)
- net -12V: now also A1.4 (-12V)
- net GND: now also A1.2 (GND)
Other:
- moved on the sheet: J5, R10, R6

Commit message: ExModule layout
Parts:
- removed unit 2 of U1
- added SW1: RESET, Button_Switch_THT:SW_Tactile_SPST_Angled_PTS645Vx39-2LFS, symbol Switch:SW_Push
- A1: footprint (none) -> BulkyMIDI-32:ExPower
- FB1: footprint Inductor_THT:L_Axial_L7.0mm_D3.3mm_P10.16mm_Horizontal_Fastron_MICC -> BulkyMIDI-32:L_Axial_L7.0mm_D3.3mm_P10.16mm_Horizontal_Fastron_MICC
Connections:
- net GND: now also SW1.1
- net RESET renamed RESET_SW
- net RESET_SW: now also SW1.2; no longer J2.26 (~RESET)
- new net ~RESET: J2.26 (~RESET)
- no-connect marks 14 -> 13

Commit message: Add ExModule panel
Parts:
- J6: footprint BulkyMIDI-32:Play_Panel -> BulkyMIDI-32:ExModule_Panel
Other:
- note added: "I don't really have a specific idea for\nhow to add +12V and -12V, so for now\nthis is just a bunch of pins for soldering\nsomething onto."
- note added: "LEDs D1, D2 as well as SW1 will be duplicated\non panel, you should only install them in one place."
- note added: "NB!"
- note added: "Not sure if this is the way to do it, or even if it\nhas been implemented correctly as to how it\nused to be done. If all fails try without it, or just\na wire."
- note added: "R4/R5 values must be adjusted to type of LED used,\nthe modern bright ones needs a substantially larger\nvalue than this (try 2k2 or 3k3 for a clear modern one)."
- moved on the sheet: A1, C1, C6, C7, D1, D2, D3, D4, J1, J2, J3, J4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
