File: faceplates/BulkyMIDI-32 ExModule FP1/BulkyMIDI-32 ExModule FP1.kicad_pcb (KiCad board)
At the start: 2 copper layers, 100 x 23.2 mm, 5 parts, among them M1 Mounting_Pin, M2 Mounting_Pin, M3 Mounting_Pin, M4 Mounting_Pin

Commit message: Power switch faceplate
Other:
- board text added: "JLCJLCJLCJLC"
- board text added: "WayWayWay"
Changed lines of the file:
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@@
   (general
     (thickness 1.6)
-    (drawings 11)
+    (drawings 13)
     (tracks 0)
     (zones 0)
@@
       (effects (font (size 1.524 1.524) (thickness 0.3)))
     )
-    (fp_poly (pts (xy -8.975176 -1.017017) (xy -10.602403 -1.017017) (xy -10.602403 -0.203403) (xy -9.788789 -0.203403)
-      (xy -9.788789 0.203404) (xy -10.602403 0.203404) (xy -10.602403 1.017017) (xy -8.975176 1.017017)
-      (xy -8.975176 1.423824) (xy -11.365165 1.423824) (xy -11.365165 -1.423823) (xy -8.975176 -1.423823)
-      (xy -8.975176 -1.017017)) (layer F.SilkS) (width 0.01))
+    (fp_poly (pts (xy 11.365165 -1.017017) (xy 9.737938 -1.017017) (xy 9.737938 -0.203403) (xy 10.551551 -0.203403)
+      (xy 10.551551 0.203404) (xy 9.737938 0.203404) (xy 9.737938 1.017017) (xy 11.365165 1.017017)
+      (xy 11.365165 1.423824) (xy 8.924324 1.423824) (xy 8.924324 -1.423823) (xy 11.365165 -1.423823)
+      (xy 11.365165 -1.017017)) (layer F.SilkS) (width 0.01))
+    (fp_poly (pts (xy 6.89029 1.017017) (xy 8.517517 1.017017) (xy 8.517517 1.423824) (xy 6.076676 1.423824)
+      (xy 6.076676 -1.423823) (xy 6.89029 -1.423823) (xy 6.89029 1.017017)) (layer F.SilkS) (width 0.01))
+    (fp_poly (pts (xy 4.042642 1.017017) (xy 4.856256 1.017017) (xy 4.856256 -1.423823) (xy 5.66987 -1.423823)
+      (xy 5.66987 1.017017) (xy 5.263063 1.017017) (xy 5.263063 1.423824) (xy 3.635836 1.423824)
+      (xy 3.635836 1.017017) (xy 3.229029 1.017017) (xy 3.229029 -1.423823) (xy 4.042642 -1.423823)
+      (xy 4.042642 1.017017)) (layer F.SilkS) (width 0.01))
+    (fp_poly (pts (xy 2.008608 -1.017017) (xy 2.415415 -1.017017) (xy 2.415415 -0.61021) (xy 2.822222 -0.61021)
+      (xy 2.822222 0.610211) (xy 2.415415 0.610211) (xy 2.415415 1.017017) (xy 2.008608 1.017017)
+      (xy 2.008608 1.423824) (xy 0.381381 1.423824) (xy 0.381381 -1.017017) (xy 1.194995 -1.017017)
+      (xy 1.194995 1.017017) (xy 1.601801 1.017017) (xy 1.601801 0.610211) (xy 2.008608 0.610211)
+      (xy 2.008608 -0.61021) (xy 1.601801 -0.61021) (xy 1.601801 -1.017017) (xy 1.194995 -1.017017)
+      (xy 0.381381 -1.017017) (xy 0.381381 -1.423823) (xy 2.008608 -1.423823) (xy 2.008608 -1.017017)) (layer F.SilkS) (width 0.01))
+    (fp_poly (pts (xy -0.432233 -1.017017) (xy -0.025426 -1.017017) (xy -0.025426 1.017017) (xy -0.432233 1.017017)
+      (xy -0.432233 1.423824) (xy -2.05946 1.423824) (xy -2.05946 1.017017) (xy -2.466267 1.017017)
+      (xy -2.466267 -1.017017) (xy -2.05946 -1.017017) (xy -1.652653 -1.017017) (xy -1.652653 1.017017)
+      (xy -0.839039 1.017017) (xy -0.839039 -1.017017) (xy -1.652653 -1.017017) (xy -2.05946 -1.017017)
+      (xy -2.05946 -1.423823) (xy -0.432233 -1.423823) (xy -0.432233 -1.017017)) (layer F.SilkS) (width 0.01))
+    (fp_poly (pts (xy -4.907107 -1.017017) (xy -4.500301 -1.017017) (xy -4.500301 -0.61021) (xy -4.093494 -0.61021)
+      (xy -4.093494 -1.017017) (xy -3.686687 -1.017017) (xy -3.686687 -1.423823) (xy -2.873073 -1.423823)
+      (xy -2.873073 1.423824) (xy -3.686687 1.423824) (xy -3.686687 -0.203403) (xy -4.093494 -0.203403)
+      (xy -4.093494 0.203404) (xy -4.500301 0.203404) (xy -4.500301 -0.203403) (xy -4.907107 -0.203403)
+      (xy -4.907107 1.423824) (xy -5.720721 1.423824) (xy -5.720721 -1.423823) (xy -4.907107 -1.423823)
+      (xy -4.907107 -1.017017)) (layer F.SilkS) (width 0.01))
     (fp_poly (pts (xy -7.754755 -0.203403) (xy -6.941141 -0.203403) (xy -6.941141 -0.61021) (xy -6.127528 -0.61021)
       (xy -6.127528 -0.203403) (xy -6.534335 -0.203403) (xy -6.534335 0.203404) (xy -6.941141 0.203404)
@@
       (xy -8.161562 -0.203403) (xy -8.568369 -0.203403) (xy -8.568369 -0.61021) (xy -7.754755 -0.61021)
       (xy -7.754755 -0.203403)) (layer F.SilkS) (width 0.01))
-    (fp_poly (pts (xy -4.907107 -1.017017) (xy -4.500301 -1.017017) (xy -4.500301 -0.61021) (xy -4.093494 -0.61021)
-      (xy -4.093494 -1.017017) (xy -3.686687 -1.017017) (xy -3.686687 -1.423823) (xy -2.873073 -1.423823)
-      (xy -2.873073 1.423824) (xy -3.686687 1.423824) (xy -3.686687 -0.203403) (xy -4.093494 -0.203403)
-      (xy -4.093494 0.203404) (xy -4.500301 0.203404) (xy -4.500301 -0.203403) (xy -4.907107 -0.203403)
-      (xy -4.907107 1.423824) (xy -5.720721 1.423824) (xy -5.720721 -1.423823) (xy -4.907107 -1.423823)
-      (xy -4.907107 -1.017017)) (layer F.SilkS) (width 0.01))
-    (fp_poly (pts (xy -0.432233 -1.017017) (xy -0.025426 -1.017017) (xy -0.025426 1.017017) (xy -0.432233 1.017017)
-      (xy -0.432233 1.423824) (xy -2.05946 1.423824) (xy -2.05946 1.017017) (xy -2.466267 1.017017)
-      (xy -2.466267 -1.017017) (xy -2.05946 -1.017017) (xy -1.652653 -1.017017) (xy -1.652653 1.017017)
-      (xy -0.839039 1.017017) (xy -0.839039 -1.017017) (xy -1.652653 -1.017017) (xy -2.05946 -1.017017)
-      (xy -2.05946 -1.423823) (xy -0.432233 -1.423823) (xy -0.432233 -1.017017)) (layer F.SilkS) (width 0.01))
-    (fp_poly (pts (xy 2.008608 -1.017017) (xy 2.415415 -1.017017) (xy 2.415415 -0.61021) (xy 2.822222 -0.61021)
-      (xy 2.822222 0.610211) (xy 2.415415 0.610211) (xy 2.415415 1.017017) (xy 2.008608 1.017017)
-      (xy 2.008608 1.423824) (xy 0.381381 1.423824) (xy 0.381381 -1.017017) (xy 1.194995 -1.017017)
-      (xy 1.194995 1.017017) (xy 1.601801 1.017017) (xy 1.601801 0.610211) (xy 2.008608 0.610211)
-      (xy 2.008608 -0.61021) (xy 1.601801 -0.61021) (xy 1.601801 -1.017017) (xy 1.194995 -1.017017)
-      (xy 0.381381 -1.017017) (xy 0.381381 -1.423823) (xy 2.008608 -1.423823) (xy 2.008608 -1.017017)) (layer F.SilkS) (width 0.01))
-    (fp_poly (pts (xy 4.042642 1.017017) (xy 4.856256 1.017017) (xy 4.856256 -1.423823) (xy 5.66987 -1.423823)
-      (xy 5.66987 1.017017) (xy 5.263063 1.017017) (xy 5.263063 1.423824) (xy 3.635836 1.423824)
-      (xy 3.635836 1.017017) (xy 3.229029 1.017017) (xy 3.229029 -1.423823) (xy 4.042642 -1.423823)
-      (xy 4.042642 1.017017)) (layer F.SilkS) (width 0.01))
-    (fp_poly (pts (xy 6.89029 1.017017) (xy 8.517517 1.017017) (xy 8.517517 1.423824) (xy 6.076676 1.423824)
-      (xy 6.076676 -1.423823) (xy 6.89029 -1.423823) (xy 6.89029 1.017017)) (layer F.SilkS) (width 0.01))
-    (fp_poly (pts (xy 11.365165 -1.017017) (xy 9.737938 -1.017017) (xy 9.737938 -0.203403) (xy 10.551551 -0.203403)
-      (xy 10.551551 0.203404) (xy 9.737938 0.203404) (xy 9.737938 1.017017) (xy 11.365165 1.017017)
-      (xy 11.365165 1.423824) (xy 8.924324 1.423824) (xy 8.924324 -1.423823) (xy 11.365165 -1.423823)
-      (xy 11.365165 -1.017017)) (layer F.SilkS) (width 0.01))
+    (fp_poly (pts (xy -8.975176 -1.017017) (xy -10.602403 -1.017017) (xy -10.602403 -0.203403) (xy -9.788789 -0.203403)
+      (xy -9.788789 0.203404) (xy -10.602403 0.203404) (xy -10.602403 1.017017) (xy -8.975176 1.017017)
+      (xy -8.975176 1.423824) (xy -11.365165 1.423824) (xy -11.365165 -1.423823) (xy -8.975176 -1.423823)
+      (xy -8.975176 -1.017017)) (layer F.SilkS) (width 0.01))
   )
   (module mounting:M3_pin (layer F.Cu)
@@
       (effects (font (size 1 1) (thickness 0.15)))
     )
-    (fp_circle (center 0 0) (end 2.6 0) (layer F.CrtYd) (width 0.05))
-    (fp_circle (center 0 0) (end 2 0.8) (layer F.Fab) (width 0.1))
+    (fp_circle (center 0 0) (end 2 0.8) (layer F.Fab) (width 0.1))
+    (fp_circle (center 0 0) (end 2.6 0) (layer F.CrtYd) (width 0.05))
     (pad 1 thru_hole circle (at 0 0) (size 3.5 3.5) (drill 3.048) (layers *.Cu *.Mask)
       (net 1 GND) (solder_mask_margin 0.8))
@@
       (effects (font (size 1 1) (thickness 0.15)))
     )
-    (fp_circle (center 0 0) (end 2 0.8) (layer F.Fab) (width 0.1))
-    (fp_circle (center 0 0) (end 2.6 0) (layer F.CrtYd) (width 0.05))
+    (fp_circle (center 0 0) (end 2.6 0) (layer F.CrtYd) (width 0.05))
+    (fp_circle (center 0 0) (end 2 0.8) (layer F.Fab) (width 0.1))
     (pad 1 thru_hole circle (at 0 0) (size 3.5 3.5) (drill 3.048) (layers *.Cu *.Mask)
       (net 1 GND) (solder_mask_margin 0.8))
@@
       (effects (font (size 1 1) (thickness 0.15)))
     )
-    (fp_circle (center 0 0) (end 2.6 0) (layer F.CrtYd) (width 0.05))
-    (fp_circle (center 0 0) (end 2 0.8) (layer F.Fab) (width 0.1))
+    (fp_circle (center 0 0) (end 2 0.8) (layer F.Fab) (width 0.1))
+    (fp_circle (center 0 0) (end 2.6 0) (layer F.CrtYd) (width 0.05))
     (pad 1 thru_hole circle (at 0 0) (size 3.5 3.5) (drill 3.048) (layers *.Cu *.Mask)
       (net 1 GND) (solder_mask_margin 0.8))
@@
       (effects (font (size 1 1) (thickness 0.15)))
     )
-    (fp_circle (center 0 0) (end 2 0.8) (layer F.Fab) (width 0.1))
-    (fp_circle (center 0 0) (end 2.6 0) (layer F.CrtYd) (width 0.05))
-    (pad 1 thru_hole circle (at 0 0) (size 3.5 3.5) (drill 3.048) (layers *.Cu *.Mask)
-      (net 1 GND) (solder_mask_margin 0.8))
+    (fp_circle (center 0 0) (end 2.6 0) (layer F.CrtYd) (width 0.05))
+    (fp_circle (center 0 0) (end 2 0.8) (layer F.Fab) (width 0.1))
+    (pad 1 thru_hole circle (at 0 0) (size 3.5 3.5) (drill 3.048) (layers *.Cu *.Mask)
+      (net 1 GND) (solder_mask_margin 0.8))
+  )
+  (gr_text JLCJLCJLCJLC (at 112.985 133.009) (layer F.Fab)
+    (effects (font (size 0.9 0.9) (thickness 0.1)) (justify mirror))
+  )
+  (gr_text WayWayWay (at 170.135 133.009) (layer B.SilkS)
+    (effects (font (size 0.9 0.9) (thickness 0.1)) (justify mirror))
   )
   (gr_text RESET (at 169.665 124.373) (layer F.SilkS)
