File: faceplates/BulkyMIDI-32 Audio Switch FP1/BulkyMIDI-32 Audio Switch FP1.kicad_pcb (KiCad board)
At the start: 2 copper layers, 100 x 23.2 mm, 5 parts, among them M1 Mounting_Pin, M2 Mounting_Pin, M3 Mounting_Pin, M4 Mounting_Pin

Commit message: Add order number placeholder
Other:
- board text added: "WayWayWay"
