File: faceplates/BulkyMIDI-32 Channel FP1/BulkyMIDI-32 Channel FP1.kicad_pcb (KiCad board)
At the start: 2 copper layers, 100 x 23.2 mm, 4 parts, among them M1 Mounting_Pin, M2 Mounting_Pin, M3 Mounting_Pin, M4 Mounting_Pin

Commit message: Channel logo added to FP1, same with Play
Parts:
- added G***: LOGO, artwork:Channel, F.Cu at (141.1, 131.8)
Changed lines of the file:
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@@
     (tracks 0)
     (zones 0)
-    (modules 4)
+    (modules 5)
     (nets 2)
   )
@@
     (add_net GND)
   )
+  (module artwork:Channel locked (layer F.Cu)
+    (at 141.09 131.8025)
+    (fp_text reference G*** (at 0 0) (layer F.SilkS) hide
+      (effects (font (size 1.524 1.524) (thickness 0.3)))
+    )
+    (fp_text value LOGO (at 0.75 0) (layer F.SilkS) hide
+      (effects (font (size 1.524 1.524) (thickness 0.3)))
+    )
+    (fp_poly (pts (xy -18.713113 -1.017017) (xy -18.306307 -1.017017) (xy -18.306307 -0.61021) (xy -19.11992 -0.61021)
+      (xy -19.11992 -1.017017) (xy -19.933534 -1.017017) (xy -19.933534 1.017017) (xy -19.11992 1.017017)
+      (xy -19.11992 0.610211) (xy -18.306307 0.610211) (xy -18.306307 1.017017) (xy -18.713113 1.017017)
+      (xy -18.713113 1.423824) (xy -20.340341 1.423824) (xy -20.340341 1.017017) (xy -20.747147 1.017017)
+      (xy -20.747147 -1.017017) (xy -20.340341 -1.017017) (xy -20.340341 -1.423823) (xy -18.713113 -1.423823)
+      (xy -18.713113 -1.017017)) (layer F.SilkS) (width 0.01))
+    (fp_poly (pts (xy -17.085886 -0.203403) (xy -15.865466 -0.203403) (xy -15.865466 0.203404) (xy -15.458659 0.203404)
+      (xy -15.458659 1.423824) (xy -16.272273 1.423824) (xy -16.272273 0.203404) (xy -17.085886 0.203404)
+      (xy -17.085886 1.423824) (xy -17.8995 1.423824) (xy -17.8995 -1.017017) (xy -17.085886 -1.017017)
+      (xy -17.085886 -0.203403)) (layer F.SilkS) (width 0.01))
+    (fp_poly (pts (xy -13.017818 -0.203403) (xy -12.611011 -0.203403) (xy -12.611011 1.423824) (xy -14.645045 1.423824)
+      (xy -14.645045 1.017017) (xy -15.051852 1.017017) (xy -15.051852 0.610211) (xy -14.645045 0.610211)
+      (xy -14.238239 0.610211) (xy -14.238239 1.017017) (xy -13.424625 1.017017) (xy -13.424625 0.610211)
+      (xy -14.238239 0.610211) (xy -14.645045 0.610211) (xy -14.645045 0.203404) (xy -13.424625 0.203404)
+      (xy -13.424625 -0.203403) (xy -14.645045 -0.203403) (xy -14.645045 -0.61021) (xy -13.017818 -0.61021)
+      (xy -13.017818 -0.203403)) (layer F.SilkS) (width 0.01))
+    (fp_poly (pts (xy -10.170171 -0.203403) (xy -9.763364 -0.203403) (xy -9.763364 1.423824) (xy -10.576977 1.423824)
+      (xy -10.576977 -0.203403) (xy -11.390591 -0.203403) (xy -11.390591 1.423824) (xy -12.204205 1.423824)
+      (xy -12.204205 -0.61021) (xy -10.170171 -0.61021) (xy -10.170171 -0.203403)) (layer F.SilkS) (width 0.01))
+    (fp_poly (pts (xy -7.322523 -0.203403) (xy -6.915716 -0.203403) (xy -6.915716 1.423824) (xy -7.72933 1.423824)
+      (xy -7.72933 -0.203403) (xy -8.542943 -0.203403) (xy -8.542943 1.423824) (xy -9.356557 1.423824)
+      (xy -9.356557 -0.61021) (xy -7.322523 -0.61021) (xy -7.322523 -0.203403)) (layer F.SilkS) (width 0.01))
+    (fp_poly (pts (xy -4.474875 -0.203403) (xy -4.068068 -0.203403) (xy -4.068068 0.610211) (xy -5.695296 0.610211)
+      (xy -5.695296 1.017017) (xy -4.474875 1.017017) (xy -4.474875 1.423824) (xy -6.102102 1.423824)
+      (xy -6.102102 1.017017) (xy -6.508909 1.017017) (xy -6.508909 -0.203403) (xy -6.102102 -0.203403)
+      (xy -5.695296 -0.203403) (xy -5.695296 0.203404) (xy -4.881682 0.203404) (xy -4.881682 -0.203403)
+      (xy -5.695296 -0.203403) (xy -6.102102 -0.203403) (xy -6.102102 -0.61021) (xy -4.474875 -0.61021)
+      (xy -4.474875 -0.203403)) (layer F.SilkS) (width 0.01))
+    (fp_poly (pts (xy -2.440841 1.017017) (xy -2.034034 1.017017) (xy -2.034034 1.423824) (xy -3.661262 1.423824)
+      (xy -3.661262 1.017017) (xy -3.254455 1.017017) (xy -3.254455 -0.61021) (xy -3.661262 -0.61021)
+      (xy -3.661262 -1.017017) (xy -2.440841 -1.017017) (xy -2.440841 1.017017)) (layer F.SilkS) (width 0.01))
+    (fp_poly (pts (xy 2.44084 -1.017017) (xy 2.847647 -1.017017) (xy 2.847647 -0.61021) (xy 3.254454 -0.61021)
+      (xy 3.254454 -1.017017) (xy 3.661261 -1.017017) (xy 3.661261 -1.423823) (xy 4.474875 -1.423823)
+      (xy 4.474875 1.423824) (xy 3.661261 1.423824) (xy 3.661261 -0.203403) (xy 3.254454 -0.203403)
+      (xy 3.254454 0.203404) (xy 2.847647 0.203404) (xy 2.847647 -0.203403) (xy 2.44084 -0.203403)
+      (xy 2.44084 1.423824) (xy 1.627227 1.423824) (xy 1.627227 -1.423823) (xy 2.44084 -1.423823)
+      (xy 2.44084 -1.017017)) (layer F.SilkS) (width 0.01))
+    (fp_poly (pts (xy 6.915715 -0.203403) (xy 7.322522 -0.203403) (xy 7.322522 1.017017) (xy 6.915715 1.017017)
+      (xy 6.915715 1.423824) (xy 5.288488 1.423824) (xy 5.288488 1.017017) (xy 4.881681 1.017017)
+      (xy 4.881681 -0.203403) (xy 5.288488 -0.203403) (xy 5.695295 -0.203403) (xy 5.695295 1.017017)
+      (xy 6.508909 1.017017) (xy 6.508909 -0.203403) (xy 5.695295 -0.203403) (xy 5.288488 -0.203403)
+      (xy 5.288488 -0.61021) (xy 6.915715 -0.61021) (xy 6.915715 -0.203403)) (layer F.SilkS) (width 0.01))
+    (fp_poly (pts (xy 9.763363 -0.203403) (xy 10.17017 -0.203403) (xy 10.17017 1.423824) (xy 9.356556 1.423824)
+      (xy 9.356556 -0.203403) (xy 8.542943 -0.203403) (xy 8.542943 1.423824) (xy 7.729329 1.423824)
+      (xy 7.729329 -0.61021) (xy 9.763363 -0.61021) (xy 9.763363 -0.203403)) (layer F.SilkS) (width 0.01))
+    (fp_poly (pts (xy 11.797397 1.017017) (xy 12.204204 1.017017) (xy 12.204204 1.423824) (xy 10.576977 1.423824)
+      (xy 10.576977 1.017017) (xy 10.983783 1.017017) (xy 10.983783 0.203404) (xy 10.576977 0.203404)
+      (xy 10.576977 -0.203403) (xy 11.797397 -0.203403) (xy 11.797397 1.017017)) (layer F.SilkS) (width 0.01))
+    (fp_poly (pts (xy 14.238238 -0.61021) (xy 15.051851 -0.61021) (xy 15.051851 -0.203403) (xy 14.238238 -0.203403)
+      (xy 14.238238 1.017017) (xy 15.051851 1.017017) (xy 15.051851 1.423824) (xy 13.831431 1.423824)
+      (xy 13.831431 1.017017) (xy 13.424624 1.017017) (xy 13.424624 -0.203403) (xy 12.611011 -0.203403)
+      (xy 12.611011 -0.61021) (xy 13.424624 -0.61021) (xy 13.424624 -1.017017) (xy 14.238238 -1.017017)
+      (xy 14.238238 -0.61021)) (layer F.SilkS) (width 0.01))
+    (fp_poly (pts (xy 17.492692 -0.203403) (xy 17.899499 -0.203403) (xy 17.899499 1.017017) (xy 17.492692 1.017017)
+      (xy 17.492692 1.423824) (xy 15.865465 1.423824) (xy 15.865465 1.017017) (xy 15.458658 1.017017)
+      (xy 15.458658 -0.203403) (xy 15.865465 -0.203403) (xy 16.272272 -0.203403) (xy 16.272272 1.017017)
+      (xy 17.085886 1.017017) (xy 17.085886 -0.203403) (xy 16.272272 -0.203403) (xy 15.865465 -0.203403)
+      (xy 15.865465 -0.61021) (xy 17.492692 -0.61021) (xy 17.492692 -0.203403)) (layer F.SilkS) (width 0.01))
+    (fp_poly (pts (xy 20.34034 -0.203403) (xy 20.747147 -0.203403) (xy 20.747147 0.203404) (xy 19.933533 0.203404)
+      (xy 19.933533 -0.203403) (xy 19.11992 -0.203403) (xy 19.11992 1.423824) (xy 18.306306 1.423824)
+      (xy 18.306306 -0.61021) (xy 20.34034 -0.61021) (xy 20.34034 -0.203403)) (layer F.SilkS) (width 0.01))
+    (fp_poly (pts (xy 11.797397 -0.61021) (xy 10.983783 -0.61021) (xy 10.983783 -1.017017) (xy 11.797397 -1.017017)
+      (xy 11.797397 -0.61021)) (layer F.SilkS) (width 0.01))
+  )
   (module mounting:M3_pin (layer F.Cu)
     (at 99.815 129.199)
@@
       (effects (font (size 1 1) (thickness 0.15)))
     )
-    (fp_circle (center 0 0) (end 2.6 0) (layer F.CrtYd) (width 0.05))
-    (fp_circle (center 0 0) (end 2 0.8) (layer F.Fab) (width 0.1))
+    (fp_circle (center 0 0) (end 2 0.8) (layer F.Fab) (width 0.1))
+    (fp_circle (center 0 0) (end 2.6 0) (layer F.CrtYd) (width 0.05))
     (pad 1 thru_hole circle (at 0 0) (size 3.5 3.5) (drill 3.048) (layers *.Cu *.Mask)
       (net 1 GND) (solder_mask_margin 0.8))
@@
       (effects (font (size 1 1) (thickness 0.15)))
     )
-    (fp_circle (center 0 0) (end 2 0.8) (layer F.Fab) (width 0.1))
-    (fp_circle (center 0 0) (end 2.6 0) (layer F.CrtYd) (width 0.05))
+    (fp_circle (center 0 0) (end 2.6 0) (layer F.CrtYd) (width 0.05))
+    (fp_circle (center 0 0) (end 2 0.8) (layer F.Fab) (width 0.1))
     (pad 1 thru_hole circle (at 0 0) (size 3.5 3.5) (drill 3.048) (layers *.Cu *.Mask)
       (net 1 GND) (solder_mask_margin 0.8))
@@
       (effects (font (size 1 1) (thickness 0.15)))
     )
-    (fp_circle (center 0 0) (end 2.6 0) (layer F.CrtYd) (width 0.05))
-    (fp_circle (center 0 0) (end 2 0.8) (layer F.Fab) (width 0.1))
+    (fp_circle (center 0 0) (end 2 0.8) (layer F.Fab) (width 0.1))
+    (fp_circle (center 0 0) (end 2.6 0) (layer F.CrtYd) (width 0.05))
     (pad 1 thru_hole circle (at 0 0) (size 3.5 3.5) (drill 3.048) (layers *.Cu *.Mask)
       (net 1 GND) (solder_mask_margin 0.8))
@@
       (effects (font (size 1 1) (thickness 0.15)))
     )
-    (fp_circle (center 0 0) (end 2 0.8) (layer F.Fab) (width 0.1))
-    (fp_circle (center 0 0) (end 2.6 0) (layer F.CrtYd) (width 0.05))
-    (pad 1 thru_hole circle (at 0 0) (size 3.5 3.5) (drill 3.048) (layers *.Cu *.Mask)
-      (net 1 GND) (solder_mask_margin 0.8))
+    (fp_circle (center 0 0) (end 2.6 0) (layer F.CrtYd) (width 0.05))
+    (fp_circle (center 0 0) (end 2 0.8) (layer F.Fab) (width 0.1))
+    (pad 1 thru_hole circle (at 0 0) (size 3.5 3.5) (drill 3.048) (layers *.Cu *.Mask)
+      (net 1 GND) (solder_mask_margin 0.8))

Commit message: Add order number placeholder
Other:
- board text added: "JLCJLCJLCJLC"
- board text added: "WayWayWay"
