File: faceplates/BulkyMIDI-32 Dexed FP4/BulkyMIDI-32 Dexed FP4.kicad_pcb (KiCad board)
At the start: 2 copper layers, 100 x 35 mm, 5 parts, among them M1 Mounting_Pin, M2 Mounting_Pin, M3 Mounting_Pin, M4 Mounting_Pin

Commit message: Add order number placeholder
Other:
- board text added: "JLCJLCJLCJLC"
Changed lines of the file:
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@@
   (general
     (thickness 1.6)
-    (drawings 24)
+    (drawings 25)
     (tracks 0)
     (zones 0)
@@
       (effects (font (size 1.524 1.524) (thickness 0.3)))
     )
-    (fp_poly (pts (xy 6.076677 -1.017017) (xy 6.483484 -1.017017) (xy 6.483484 -0.61021) (xy 6.890291 -0.61021)
-      (xy 6.890291 0.610211) (xy 6.483484 0.610211) (xy 6.483484 1.017017) (xy 6.076677 1.017017)
-      (xy 6.076677 1.423824) (xy 4.44945 1.423824) (xy 4.44945 -1.017017) (xy 5.263063 -1.017017)
-      (xy 5.263063 1.017017) (xy 5.66987 1.017017) (xy 5.66987 0.610211) (xy 6.076677 0.610211)
-      (xy 6.076677 -0.61021) (xy 5.66987 -0.61021) (xy 5.66987 -1.017017) (xy 5.263063 -1.017017)
-      (xy 4.44945 -1.017017) (xy 4.44945 -1.423823) (xy 6.076677 -1.423823) (xy 6.076677 -1.017017)) (layer F.SilkS) (width 0.01))
-    (fp_poly (pts (xy 4.042643 -1.017017) (xy 2.415416 -1.017017) (xy 2.415416 -0.203403) (xy 3.229029 -0.203403)
-      (xy 3.229029 0.203404) (xy 2.415416 0.203404) (xy 2.415416 1.017017) (xy 4.042643 1.017017)
-      (xy 4.042643 1.423824) (xy 1.601802 1.423824) (xy 1.601802 -1.423823) (xy 4.042643 -1.423823)
-      (xy 4.042643 -1.017017)) (layer F.SilkS) (width 0.01))
+    (fp_poly (pts (xy -5.313914 -1.017017) (xy -4.907107 -1.017017) (xy -4.907107 -0.61021) (xy -4.5003 -0.61021)
+      (xy -4.5003 0.610211) (xy -4.907107 0.610211) (xy -4.907107 1.017017) (xy -5.313914 1.017017)
+      (xy -5.313914 1.423824) (xy -6.915715 1.423824) (xy -6.915715 -1.017017) (xy -6.127527 -1.017017)
+      (xy -6.127527 1.017017) (xy -5.720721 1.017017) (xy -5.720721 0.610211) (xy -5.313914 0.610211)
+      (xy -5.313914 -0.61021) (xy -5.720721 -0.61021) (xy -5.720721 -1.017017) (xy -6.127527 -1.017017)
+      (xy -6.915715 -1.017017) (xy -6.915715 -1.423823) (xy -5.313914 -1.423823) (xy -5.313914 -1.017017)) (layer F.SilkS) (width 0.01))
+    (fp_poly (pts (xy -1.652652 -1.017017) (xy -3.27988 -1.017017) (xy -3.27988 -0.203403) (xy -2.466266 -0.203403)
+      (xy -2.466266 0.203404) (xy -3.27988 0.203404) (xy -3.27988 1.017017) (xy -1.652652 1.017017)
+      (xy -1.652652 1.423824) (xy -4.093493 1.423824) (xy -4.093493 -1.423823) (xy -1.652652 -1.423823)
+      (xy -1.652652 -1.017017)) (layer F.SilkS) (width 0.01))
     (fp_poly (pts (xy -0.432232 -0.61021) (xy 0.381382 -0.61021) (xy 0.381382 -1.423823) (xy 1.194995 -1.423823)
       (xy 1.194995 -0.61021) (xy 0.788188 -0.61021) (xy 0.788188 -0.203403) (xy 0.381382 -0.203403)
@@
       (xy -0.839039 -0.61021) (xy -1.245846 -0.61021) (xy -1.245846 -1.423823) (xy -0.432232 -1.423823)
       (xy -0.432232 -0.61021)) (layer F.SilkS) (width 0.01))
-    (fp_poly (pts (xy -1.652652 -1.017017) (xy -3.27988 -1.017017) (xy -3.27988 -0.203403) (xy -2.466266 -0.203403)
-      (xy -2.466266 0.203404) (xy -3.27988 0.203404) (xy -3.27988 1.017017) (xy -1.652652 1.017017)
-      (xy -1.652652 1.423824) (xy -4.093493 1.423824) (xy -4.093493 -1.423823) (xy -1.652652 -1.423823)
-      (xy -1.652652 -1.017017)) (layer F.SilkS) (width 0.01))
-    (fp_poly (pts (xy -5.313914 -1.017017) (xy -4.907107 -1.017017) (xy -4.907107 -0.61021) (xy -4.5003 -0.61021)
-      (xy -4.5003 0.610211) (xy -4.907107 0.610211) (xy -4.907107 1.017017) (xy -5.313914 1.017017)
-      (xy -5.313914 1.423824) (xy -6.915715 1.423824) (xy -6.915715 -1.017017) (xy -6.127527 -1.017017)
-      (xy -6.127527 1.017017) (xy -5.720721 1.017017) (xy -5.720721 0.610211) (xy -5.313914 0.610211)
-      (xy -5.313914 -0.61021) (xy -5.720721 -0.61021) (xy -5.720721 -1.017017) (xy -6.127527 -1.017017)
-      (xy -6.915715 -1.017017) (xy -6.915715 -1.423823) (xy -5.313914 -1.423823) (xy -5.313914 -1.017017)) (layer F.SilkS) (width 0.01))
+    (fp_poly (pts (xy 4.042643 -1.017017) (xy 2.415416 -1.017017) (xy 2.415416 -0.203403) (xy 3.229029 -0.203403)
+      (xy 3.229029 0.203404) (xy 2.415416 0.203404) (xy 2.415416 1.017017) (xy 4.042643 1.017017)
+      (xy 4.042643 1.423824) (xy 1.601802 1.423824) (xy 1.601802 -1.423823) (xy 4.042643 -1.423823)
+      (xy 4.042643 -1.017017)) (layer F.SilkS) (width 0.01))
+    (fp_poly (pts (xy 6.076677 -1.017017) (xy 6.483484 -1.017017) (xy 6.483484 -0.61021) (xy 6.890291 -0.61021)
+      (xy 6.890291 0.610211) (xy 6.483484 0.610211) (xy 6.483484 1.017017) (xy 6.076677 1.017017)
+      (xy 6.076677 1.423824) (xy 4.44945 1.423824) (xy 4.44945 -1.017017) (xy 5.263063 -1.017017)
+      (xy 5.263063 1.017017) (xy 5.66987 1.017017) (xy 5.66987 0.610211) (xy 6.076677 0.610211)
+      (xy 6.076677 -0.61021) (xy 5.66987 -0.61021) (xy 5.66987 -1.017017) (xy 5.263063 -1.017017)
+      (xy 4.44945 -1.017017) (xy 4.44945 -1.423823) (xy 6.076677 -1.423823) (xy 6.076677 -1.017017)) (layer F.SilkS) (width 0.01))
   )
   (module mounting:M3_pin (layer F.Cu)
@@
       (effects (font (size 1 1) (thickness 0.15)))
     )
-    (fp_circle (center 0 0) (end 2 0.8) (layer F.Fab) (width 0.1))
-    (fp_circle (center 0 0) (end 2.6 0) (layer F.CrtYd) (width 0.05))
+    (fp_circle (center 0 0) (end 2.6 0) (layer F.CrtYd) (width 0.05))
+    (fp_circle (center 0 0) (end 2 0.8) (layer F.Fab) (width 0.1))
     (pad 1 thru_hole circle (at 0 0) (size 3.5 3.5) (drill 3.048) (layers *.Cu *.Mask)
       (net 1 GND) (solder_mask_margin 0.8))
@@
       (effects (font (size 1 1) (thickness 0.15)))
     )
-    (fp_circle (center 0 0) (end 2.6 0) (layer F.CrtYd) (width 0.05))
-    (fp_circle (center 0 0) (end 2 0.8) (layer F.Fab) (width 0.1))
+    (fp_circle (center 0 0) (end 2 0.8) (layer F.Fab) (width 0.1))
+    (fp_circle (center 0 0) (end 2.6 0) (layer F.CrtYd) (width 0.05))
     (pad 1 thru_hole circle (at 0 0) (size 3.5 3.5) (drill 3.048) (layers *.Cu *.Mask)
       (net 1 GND) (solder_mask_margin 0.8))
@@
       (effects (font (size 1 1) (thickness 0.15)))
     )
-    (fp_circle (center 0 0) (end 2 0.8) (layer F.Fab) (width 0.1))
-    (fp_circle (center 0 0) (end 2.6 0) (layer F.CrtYd) (width 0.05))
+    (fp_circle (center 0 0) (end 2.6 0) (layer F.CrtYd) (width 0.05))
+    (fp_circle (center 0 0) (end 2 0.8) (layer F.Fab) (width 0.1))
     (pad 1 thru_hole circle (at 0 0) (size 3.5 3.5) (drill 3.048) (layers *.Cu *.Mask)
       (net 1 GND) (solder_mask_margin 0.8))
@@
       (effects (font (size 1 1) (thickness 0.15)))
     )
-    (fp_circle (center 0 0) (end 2.6 0) (layer F.CrtYd) (width 0.05))
-    (fp_circle (center 0 0) (end 2 0.8) (layer F.Fab) (width 0.1))
-    (pad 1 thru_hole circle (at 0 0) (size 3.5 3.5) (drill 3.048) (layers *.Cu *.Mask)
-      (net 1 GND) (solder_mask_margin 0.8))
+    (fp_circle (center 0 0) (end 2 0.8) (layer F.Fab) (width 0.1))
+    (fp_circle (center 0 0) (end 2.6 0) (layer F.CrtYd) (width 0.05))
+    (pad 1 thru_hole circle (at 0 0) (size 3.5 3.5) (drill 3.048) (layers *.Cu *.Mask)
+      (net 1 GND) (solder_mask_margin 0.8))
+  )
+  (gr_text WayWayWay (at 169.665 133.009) (layer B.SilkS)
+    (effects (font (size 0.9 0.9) (thickness 0.1)) (justify mirror))
+  )
+  (gr_text JLCJLCJLCJLC (at 112.515 133.009) (layer F.Fab)
+    (effects (font (size 0.9 0.9) (thickness 0.1)) (justify mirror))
   )
   (gr_line (start 153.055 131.652) (end 129.125 131.652) (layer Edge.Cuts) (width 0.15))
@@
     (effects (font (size 0.8 0.8) (thickness 0.1)))
   )
-  (gr_text WayWayWay (at 96.3352 143.7786) (layer B.SilkS)
-    (effects (font (size 1 1) (thickness 0.15)) (justify mirror))
-  )
   (gr_circle (center 108.578 117.879) (end 110.478 117.879) (layer Edge.Cuts) (width 0.05))
