File: faceplates/BulkyMIDI-32 Internal FP1/BulkyMIDI-32 Internal FP1.kicad_pcb (KiCad board)
At the start: 2 copper layers, 101.5 x 25.7 mm, 11 parts, among them M1 Mounting_Pin, M10 Mounting_Pad, M2 Mounting_Pin, M3 Mounting_Pin, M4 Mounting_Pin, M5 Mounting_Pad, M6 Mounting_Pad, M7 Mounting_Pad, M8 Mounting_Pad, M9 Mounting_Pad

Commit message: Add order number placeholder
Other:
- board text added: "WayWayWay"
