File: faceplates/BulkyMIDI-32 Module FP1/BulkyMIDI-32 Module FP1.kicad_pcb (KiCad board)
At the start: 2 copper layers, 100 x 44.7 mm, 5 parts, among them M1 Mounting_Pin, M2 Mounting_Pin, M3 Mounting_Pin, M4 Mounting_Pin

Commit message: Moved extras LEDs to match FP1
Other:
- outline, holes or cut-outs redrawn

Commit message: Remove temporary file
Other:
- outline, holes or cut-outs redrawn
- board text added: "BulkyMIDI-32 Module FP1 (rev. B) github.com/tebl"
- board text removed: "BulkyMIDI-32 Module FP1 (rev. A) github.com/tebl"
Changed lines of the file:
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@@
   )
   (gr_circle (center 117.338 121.579) (end 119.238 121.579) (layer Edge.Cuts) (width 0.05))
-  (gr_line (start 124.58 137.475) (end 124.58 117.769) (layer Edge.Cuts) (width 0.05))
+  (gr_line (start 124.58 137.475) (end 124.58 118.169) (layer Edge.Cuts) (width 0.05))
   (gr_line (start 157.6 137.475) (end 124.58 137.475) (layer Edge.Cuts) (width 0.05))
-  (gr_line (start 157.6 117.769) (end 157.6 137.475) (layer Edge.Cuts) (width 0.05))
-  (gr_line (start 124.58 117.769) (end 157.6 117.769) (layer Edge.Cuts) (width 0.05))
+  (gr_line (start 157.6 118.169) (end 157.6 137.475) (layer Edge.Cuts) (width 0.05))
+  (gr_line (start 124.58 118.169) (end 157.6 118.169) (layer Edge.Cuts) (width 0.05))
   (gr_circle (center 169.792 121.579) (end 173.542 121.579) (layer Edge.Cuts) (width 0.05))
-  (gr_text "BulkyMIDI-32\nModule FP1 (rev. A)\ngithub.com/tebl" (at 94.1 122.849 270) (layer B.SilkS)
+  (gr_text "BulkyMIDI-32\nModule FP1 (rev. B)\ngithub.com/tebl" (at 94.1 122.849 270) (layer B.SilkS)
     (effects (font (size 0.8 0.8) (thickness 0.1)) (justify mirror))
   )

Commit message: Adjust INPUT1/INPUT2 slightly to the right
Other:
- outline, holes or cut-outs redrawn
- board text added: "BulkyMIDI-32 Module FP1 (rev. C) github.com/tebl"
- board text removed: "BulkyMIDI-32 Module FP1 (rev. B) github.com/tebl"
Changed lines of the file:
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@@
   (gr_circle (center 117.338 153.329) (end 119.238 153.329) (layer Edge.Cuts) (width 0.05))
   (gr_circle (center 108.578 153.329) (end 110.478 153.329) (layer Edge.Cuts) (width 0.05))
-  (gr_text "INPUT 2" (at 179.914 152.948) (layer F.SilkS)
+  (gr_text "INPUT 2" (at 180.114 152.948) (layer F.SilkS)
     (effects (font (size 0.8 0.8) (thickness 0.1)))
   )
-  (gr_text "INPUT 1" (at 165.055 152.948) (layer F.SilkS)
+  (gr_text "INPUT 1" (at 165.255 152.948) (layer F.SilkS)
     (effects (font (size 0.8 0.8) (thickness 0.1)))
   )
-  (gr_circle (center 165.055 147.874) (end 169.055 147.874) (layer Edge.Cuts) (width 0.05))
-  (gr_circle (center 179.914 147.874) (end 183.914 147.874) (layer Edge.Cuts) (width 0.05))
+  (gr_circle (center 165.255 147.874) (end 169.255 147.874) (layer Edge.Cuts) (width 0.05))
+  (gr_circle (center 180.114 147.874) (end 184.114 147.874) (layer Edge.Cuts) (width 0.05))
   (gr_line (start 91.09 153.874) (end 191.09 153.874) (layer Dwgs.User) (width 0.05))
   (gr_line (start 191.09 153.874) (end 191.09 155.674) (layer Dwgs.User) (width 0.05))
@@
   (gr_line (start 124.58 118.169) (end 157.6 118.169) (layer Edge.Cuts) (width 0.05))
   (gr_circle (center 169.792 121.579) (end 173.542 121.579) (layer Edge.Cuts) (width 0.05))
-  (gr_text "BulkyMIDI-32\nModule FP1 (rev. B)\ngithub.com/tebl" (at 94.1 122.849 270) (layer B.SilkS)
+  (gr_text "BulkyMIDI-32\nModule FP1 (rev. C)\ngithub.com/tebl" (at 94.1 122.849 270) (layer B.SilkS)
     (effects (font (size 0.8 0.8) (thickness 0.1)) (justify mirror))
   )

Commit message: Add order number placeholder
Other:
- board text added: "JLCJLCJLCJLC"
- board text added: "WayWayWay"
