File: faceplates/BulkyMIDI-32 VU SIDi FP1/BulkyMIDI-32 VU SIDi FP1.kicad_pcb (KiCad board)
At the start: 2 copper layers, 100 x 23.2 mm, 5 parts, among them M1 Mounting_Pin, M2 Mounting_Pin, M3 Mounting_Pin, M4 Mounting_Pin

Commit message: Add order number placeholder
Other:
- board text added: "JLCJLCJLCJLC"
- board text added: "WayWayWay"
Changed lines of the file:
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@@
   (general
     (thickness 1.6)
-    (drawings 27)
+    (drawings 29)
     (tracks 0)
     (zones 0)
@@
       (effects (font (size 1.524 1.524) (thickness 0.3)))
     )
-    (fp_poly (pts (xy 8.746346 -0.61021) (xy 7.932732 -0.61021) (xy 7.932732 -1.017017) (xy 8.746346 -1.017017)
-      (xy 8.746346 -0.61021)) (layer F.SilkS) (width 0.01))
-    (fp_poly (pts (xy 8.746346 1.017017) (xy 9.153153 1.017017) (xy 9.153153 1.423824) (xy 7.525926 1.423824)
-      (xy 7.525926 1.017017) (xy 7.932732 1.017017) (xy 7.932732 0.203404) (xy 7.525926 0.203404)
-      (xy 7.525926 -0.203403) (xy 8.746346 -0.203403) (xy 8.746346 1.017017)) (layer F.SilkS) (width 0.01))
-    (fp_poly (pts (xy 6.305505 -1.017017) (xy 6.712312 -1.017017) (xy 6.712312 -0.61021) (xy 7.119119 -0.61021)
-      (xy 7.119119 0.610211) (xy 6.712312 0.610211) (xy 6.712312 1.017017) (xy 6.305505 1.017017)
-      (xy 6.305505 1.423824) (xy 4.678278 1.423824) (xy 4.678278 -1.017017) (xy 5.491892 -1.017017)
-      (xy 5.491892 1.017017) (xy 5.898698 1.017017) (xy 5.898698 0.610211) (xy 6.305505 0.610211)
-      (xy 6.305505 -0.61021) (xy 5.898698 -0.61021) (xy 5.898698 -1.017017) (xy 5.491892 -1.017017)
-      (xy 4.678278 -1.017017) (xy 4.678278 -1.423823) (xy 6.305505 -1.423823) (xy 6.305505 -1.017017)) (layer F.SilkS) (width 0.01))
-    (fp_poly (pts (xy 4.271471 -1.017017) (xy 3.864664 -1.017017) (xy 3.864664 1.017017) (xy 4.271471 1.017017)
-      (xy 4.271471 1.423824) (xy 2.644244 1.423824) (xy 2.644244 1.017017) (xy 3.051051 1.017017)
-      (xy 3.051051 -1.017017) (xy 2.644244 -1.017017) (xy 2.644244 -1.423823) (xy 4.271471 -1.423823)
-      (xy 4.271471 -1.017017)) (layer F.SilkS) (width 0.01))
+    (fp_poly (pts (xy -8.33954 0.610211) (xy -7.525926 0.610211) (xy -7.525926 -1.423823) (xy -6.712313 -1.423823)
+      (xy -6.712313 0.610211) (xy -7.119119 0.610211) (xy -7.119119 1.017017) (xy -7.525926 1.017017)
+      (xy -7.525926 1.423824) (xy -8.33954 1.423824) (xy -8.33954 1.017017) (xy -8.746347 1.017017)
+      (xy -8.746347 0.610211) (xy -9.153153 0.610211) (xy -9.153153 -1.423823) (xy -8.33954 -1.423823)
+      (xy -8.33954 0.610211)) (layer F.SilkS) (width 0.01))
+    (fp_poly (pts (xy -5.491892 1.017017) (xy -4.678279 1.017017) (xy -4.678279 -1.423823) (xy -3.864665 -1.423823)
+      (xy -3.864665 1.017017) (xy -4.271472 1.017017) (xy -4.271472 1.423824) (xy -5.898699 1.423824)
+      (xy -5.898699 1.017017) (xy -6.305506 1.017017) (xy -6.305506 -1.423823) (xy -5.491892 -1.423823)
+      (xy -5.491892 1.017017)) (layer F.SilkS) (width 0.01))
     (fp_poly (pts (xy 1.83063 -1.017017) (xy 2.237437 -1.017017) (xy 2.237437 -0.61021) (xy 1.423823 -0.61021)
       (xy 1.423823 -1.017017) (xy 0.61021 -1.017017) (xy 0.61021 -0.203403) (xy 1.83063 -0.203403)
@@
       (xy -0.203404 -1.017017) (xy 0.203403 -1.017017) (xy 0.203403 -1.423823) (xy 1.83063 -1.423823)
       (xy 1.83063 -1.017017)) (layer F.SilkS) (width 0.01))
-    (fp_poly (pts (xy -5.491892 1.017017) (xy -4.678279 1.017017) (xy -4.678279 -1.423823) (xy -3.864665 -1.423823)
-      (xy -3.864665 1.017017) (xy -4.271472 1.017017) (xy -4.271472 1.423824) (xy -5.898699 1.423824)
-      (xy -5.898699 1.017017) (xy -6.305506 1.017017) (xy -6.305506 -1.423823) (xy -5.491892 -1.423823)
-      (xy -5.491892 1.017017)) (layer F.SilkS) (width 0.01))
-    (fp_poly (pts (xy -8.33954 0.610211) (xy -7.525926 0.610211) (xy -7.525926 -1.423823) (xy -6.712313 -1.423823)
-      (xy -6.712313 0.610211) (xy -7.119119 0.610211) (xy -7.119119 1.017017) (xy -7.525926 1.017017)
-      (xy -7.525926 1.423824) (xy -8.33954 1.423824) (xy -8.33954 1.017017) (xy -8.746347 1.017017)
-      (xy -8.746347 0.610211) (xy -9.153153 0.610211) (xy -9.153153 -1.423823) (xy -8.33954 -1.423823)
-      (xy -8.33954 0.610211)) (layer F.SilkS) (width 0.01))
+    (fp_poly (pts (xy 4.271471 -1.017017) (xy 3.864664 -1.017017) (xy 3.864664 1.017017) (xy 4.271471 1.017017)
+      (xy 4.271471 1.423824) (xy 2.644244 1.423824) (xy 2.644244 1.017017) (xy 3.051051 1.017017)
+      (xy 3.051051 -1.017017) (xy 2.644244 -1.017017) (xy 2.644244 -1.423823) (xy 4.271471 -1.423823)
+      (xy 4.271471 -1.017017)) (layer F.SilkS) (width 0.01))
+    (fp_poly (pts (xy 6.305505 -1.017017) (xy 6.712312 -1.017017) (xy 6.712312 -0.61021) (xy 7.119119 -0.61021)
+      (xy 7.119119 0.610211) (xy 6.712312 0.610211) (xy 6.712312 1.017017) (xy 6.305505 1.017017)
+      (xy 6.305505 1.423824) (xy 4.678278 1.423824) (xy 4.678278 -1.017017) (xy 5.491892 -1.017017)
+      (xy 5.491892 1.017017) (xy 5.898698 1.017017) (xy 5.898698 0.610211) (xy 6.305505 0.610211)
+      (xy 6.305505 -0.61021) (xy 5.898698 -0.61021) (xy 5.898698 -1.017017) (xy 5.491892 -1.017017)
+      (xy 4.678278 -1.017017) (xy 4.678278 -1.423823) (xy 6.305505 -1.423823) (xy 6.305505 -1.017017)) (layer F.SilkS) (width 0.01))
+    (fp_poly (pts (xy 8.746346 1.017017) (xy 9.153153 1.017017) (xy 9.153153 1.423824) (xy 7.525926 1.423824)
+      (xy 7.525926 1.017017) (xy 7.932732 1.017017) (xy 7.932732 0.203404) (xy 7.525926 0.203404)
+      (xy 7.525926 -0.203403) (xy 8.746346 -0.203403) (xy 8.746346 1.017017)) (layer F.SilkS) (width 0.01))
+    (fp_poly (pts (xy 8.746346 -0.61021) (xy 7.932732 -0.61021) (xy 7.932732 -1.017017) (xy 8.746346 -1.017017)
+      (xy 8.746346 -0.61021)) (layer F.SilkS) (width 0.01))
   )
   (module mounting:M3_pin (layer F.Cu)
@@
       (effects (font (size 1 1) (thickness 0.15)))
     )
-    (fp_circle (center 0 0) (end 2.6 0) (layer F.CrtYd) (width 0.05))
-    (fp_circle (center 0 0) (end 2 0.8) (layer F.Fab) (width 0.1))
+    (fp_circle (center 0 0) (end 2 0.8) (layer F.Fab) (width 0.1))
+    (fp_circle (center 0 0) (end 2.6 0) (layer F.CrtYd) (width 0.05))
     (pad 1 thru_hole circle (at 0 0) (size 3.5 3.5) (drill 3.048) (layers *.Cu *.Mask)
       (net 1 "Net-(M1-Pad1)") (solder_mask_margin 0.8))
@@
       (effects (font (size 1 1) (thickness 0.15)))
     )
-    (fp_circle (center 0 0) (end 2 0.8) (layer F.Fab) (width 0.1))
-    (fp_circle (center 0 0) (end 2.6 0) (layer F.CrtYd) (width 0.05))
+    (fp_circle (center 0 0) (end 2.6 0) (layer F.CrtYd) (width 0.05))
+    (fp_circle (center 0 0) (end 2 0.8) (layer F.Fab) (width 0.1))
     (pad 1 thru_hole circle (at 0 0) (size 3.5 3.5) (drill 3.048) (layers *.Cu *.Mask)
       (net 1 "Net-(M1-Pad1)") (solder_mask_margin 0.8))
@@
       (effects (font (size 1 1) (thickness 0.15)))
     )
-    (fp_circle (center 0 0) (end 2.6 0) (layer F.CrtYd) (width 0.05))
-    (fp_circle (center 0 0) (end 2 0.8) (layer F.Fab) (width 0.1))
+    (fp_circle (center 0 0) (end 2 0.8) (layer F.Fab) (width 0.1))
+    (fp_circle (center 0 0) (end 2.6 0) (layer F.CrtYd) (width 0.05))
     (pad 1 thru_hole circle (at 0 0) (size 3.5 3.5) (drill 3.048) (layers *.Cu *.Mask)
       (net 1 "Net-(M1-Pad1)") (solder_mask_margin 0.8))
@@
       (effects (font (size 1 1) (thickness 0.15)))
     )
-    (fp_circle (center 0 0) (end 2 0.8) (layer F.Fab) (width 0.1))
-    (fp_circle (center 0 0) (end 2.6 0) (layer F.CrtYd) (width 0.05))
-    (pad 1 thru_hole circle (at 0 0) (size 3.5 3.5) (drill 3.048) (layers *.Cu *.Mask)
-      (net 1 "Net-(M1-Pad1)") (solder_mask_margin 0.8))
+    (fp_circle (center 0 0) (end 2.6 0) (layer F.CrtYd) (width 0.05))
+    (fp_circle (center 0 0) (end 2 0.8) (layer F.Fab) (width 0.1))
+    (pad 1 thru_hole circle (at 0 0) (size 3.5 3.5) (drill 3.048) (layers *.Cu *.Mask)
+      (net 1 "Net-(M1-Pad1)") (solder_mask_margin 0.8))
+  )
+  (gr_text WayWayWay (at 169.665 133.009) (layer B.SilkS)
+    (effects (font (size 0.9 0.9) (thickness 0.1)) (justify mirror))
+  )
+  (gr_text JLCJLCJLCJLC (at 112.515 133.009) (layer F.Fab)
+    (effects (font (size 0.9 0.9) (thickness 0.1)) (justify mirror))
   )
   (gr_circle (center 172.5225 124.754) (end 174.4225 124.754) (layer Edge.Cuts) (width 0.05))
