File: BulkyMIDI-32 Power Switch Panel/BulkyMIDI-32 Power Switch Panel.sch (KiCad schematic (older format))
At the start: 18 parts, among them J1 Switch Panel, M1 Mounting_Pin, M2 Mounting_Pin, M3 Mounting_Pin, M4 Mounting_Pin, SW1 CH1, SW2 CH2, SW3 CH3, SW4 CH4, SW5 CH5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

Commit message: Fixes panel errors and inconsistencies
Connections:
- net GND: now also SW1.1, SW2.1, SW3.1, SW4.1, SW5.1, SW6.1
- net VCC: no longer SW1.1, SW2.1, SW3.1, SW4.1, SW5.1, SW6.1
Other:
- moved on the sheet: SW1, SW2, SW3, SW4, SW5, SW6
Changed lines of the file:
@@
 Title "Power Switch (Panel)"
 Date ""
-Rev "A"
+Rev "B"
 Comp ""
-Comment1 "NB! At the moment this is functionally identical to audio switch panel."
+Comment1 ""
 Comment2 ""
 Comment3 ""
@@
 Connection ~ 4050 4375
 Wire Wire Line
-	4125 2475 4025 2475
-Wire Wire Line
-	4125 2475 4125 2400
+	4050 2475 4050 2400
 $Comp
 L power:VCC #PWR0102
 U 1 1 62828DC5
-P 4125 2400
-F 0 "#PWR0102" H 4125 2250 50  0001 C CNN
-F 1 "VCC" H 4140 2573 50  0000 C CNN
-F 2 "" H 4125 2400 50  0001 C CNN
-F 3 "" H 4125 2400 50  0001 C CNN
-	1    4125 2400
+P 4050 2400
+F 0 "#PWR0102" H 4050 2250 50  0001 C CNN
+F 1 "VCC" H 4065 2573 50  0000 C CNN
+F 2 "" H 4050 2400 50  0001 C CNN
+F 3 "" H 4050 2400 50  0001 C CNN
+	1    4050 2400
 	-1   0    0    -1
 $EndComp
@@
 L power:PWR_FLAG #FLG0101
 U 1 1 628346CB
-P 4025 2475
-F 0 "#FLG0101" H 4025 2550 50  0001 C CNN
-F 1 "PWR_FLAG" H 4025 2648 50  0001 C CNN
-F 2 "" H 4025 2475 50  0001 C CNN
-F 3 "~" H 4025 2475 50  0001 C CNN
-	1    4025 2475
-	-1   0    0    -1
-$EndComp
-Connection ~ 4025 2475
-Wire Wire Line
-	4025 2475 3950 2475
+P 4125 2475
+F 0 "#FLG0101" H 4125 2550 50  0001 C CNN
+F 1 "PWR_FLAG" H 4125 2648 50  0001 C CNN
+F 2 "" H 4125 2475 50  0001 C CNN
+F 3 "~" H 4125 2475 50  0001 C CNN
+	1    4125 2475
+	0    1    -1   0
+$EndComp
 Wire Wire Line
 	4050 2575 3950 2575
@@
 L power:PWR_FLAG #FLG0102
 U 1 1 628CF525
-P 4050 4575
-F 0 "#FLG0102" H 4050 4650 50  0001 C CNN
-F 1 "PWR_FLAG" V 4050 4702 50  0001 L CNN
-F 2 "" H 4050 4575 50  0001 C CNN
-F 3 "~" H 4050 4575 50  0001 C CNN
-	1    4050 4575
+P 4125 4375
+F 0 "#FLG0102" H 4125 4450 50  0001 C CNN
+F 1 "PWR_FLAG" V 4125 4502 50  0001 L CNN
+F 2 "" H 4125 4375 50  0001 C CNN
+F 3 "~" H 4125 4375 50  0001 C CNN
+	1    4125 4375
 	0    1    -1   0
 $EndComp
-Wire Wire Line
-	4050 4375 4050 4575
 $Comp
 L mounting:Mounting_Pin M1
@@
 Entry Bus Bus
 	7750 4950 7650 5050
-Wire Wire Line
-	4050 4575 4050 4650
-Connection ~ 4050 4575
 Connection ~ 10975 800
 $Comp
 L Switch:SW_Push SW1
 U 1 1 62CDB5FB
-P 5450 2675
-F 0 "SW1" H 5450 2960 50  0000 C CNN
-F 1 "CH1" H 5450 2869 50  0000 C CNN
-F 2 "switch_cutout:SW_PUSH_6mm" H 5450 2875 50  0001 C CNN
-F 3 "~" H 5450 2875 50  0001 C CNN
-	1    5450 2675
-	1    0    0    -1
-$EndComp
-$Comp
-L power:VCC #PWR04
-U 1 1 62CDC310
-P 5175 2600
-F 0 "#PWR04" H 5175 2450 50  0001 C CNN
-F 1 "VCC" H 5190 2773 50  0000 C CNN
-F 2 "" H 5175 2600 50  0001 C CNN
-F 3 "" H 5175 2600 50  0001 C CNN
-	1    5175 2600
-	1    0    0    -1
-$EndComp
-Wire Wire Line
-	5175 2600 5175 2675
-Wire Wire Line
-	5175 2675 5250 2675
+P 5475 2275
+F 0 "SW1" H 5475 2560 50  0000 C CNN
+F 1 "CH1" H 5475 2469 50  0000 C CNN
+F 2 "switch_cutout:SW_PUSH_6mm" H 5475 2475 50  0001 C CNN
+F 3 "~" H 5475 2475 50  0001 C CNN
+	1    5475 2275
+	1    0    0    -1
+$EndComp
+Wire Wire Line
+	5200 2275 5275 2275
 $Comp
 L Switch:SW_Push SW2
 U 1 1 62CDF85A
-P 5450 3075
-F 0 "SW2" H 5450 3360 50  0000 C CNN
-F 1 "CH2" H 5450 3269 50  0000 C CNN
-F 2 "switch_cutout:SW_PUSH_6mm" H 5450 3275 50  0001 C CNN
-F 3 "~" H 5450 3275 50  0001 C CNN
-	1    5450 3075
-	1    0    0    -1
-$EndComp
-Wire Wire Line
-	5175 3075 5250 3075
+P 5475 2675
+F 0 "SW2" H 5475 2960 50  0000 C CNN
+F 1 "CH2" H 5475 2869 50  0000 C CNN
+F 2 "switch_cutout:SW_PUSH_6mm" H 5475 2875 50  0001 C CNN
+F 3 "~" H 5475 2875 50  0001 C CNN
+	1    5475 2675
+	1    0    0    -1
+$EndComp
+Wire Wire Line
+	5200 2675 5275 2675
 $Comp
 L Switch:SW_Push SW3
 U 1 1 62CE1A42
-P 5450 3475
-F 0 "SW3" H 5450 3760 50  0000 C CNN
-F 1 "CH3" H 5450 3669 50  0000 C CNN
-F 2 "switch_cutout:SW_PUSH_6mm" H 5450 3675 50  0001 C CNN
-F 3 "~" H 5450 3675 50  0001 C CNN
-	1    5450 3475
+P 5475 3075
+F 0 "SW3" H 5475 3360 50  0000 C CNN
+F 1 "CH3" H 5475 3269 50  0000 C CNN
+F 2 "switch_cutout:SW_PUSH_6mm" H 5475 3275 50  0001 C CNN
+F 3 "~" H 5475 3275 50  0001 C CNN
+	1    5475 3075
 	1    0    0    -1
 $EndComp
@@
 L Switch:SW_Push SW4
 U 1 1 62CE1A48
-P 5450 3875
-F 0 "SW4" H 5450 4160 50  0000 C CNN
-F 1 "CH4" H 5450 4069 50  0000 C CNN
-F 2 "switch_cutout:SW_PUSH_6mm" H 5450 4075 50  0001 C CNN
-F 3 "~" H 5450 4075 50  0001 C CNN
-	1    5450 3875
+P 5475 3475
+F 0 "SW4" H 5475 3760 50  0000 C CNN
+F 1 "CH4" H 5475 3669 50  0000 C CNN
+F 2 "switch_cutout:SW_PUSH_6mm" H 5475 3675 50  0001 C CNN
+F 3 "~" H 5475 3675 50  0001 C CNN
+	1    5475 3475
 	1    0    0    -1
 $EndComp
@@
 L Switch:SW_Push SW5
 U 1 1 62CE4BA8
-P 5450 4275
-F 0 "SW5" H 5450 4560 50  0000 C CNN
-F 1 "CH5" H 5450 4469 50  0000 C CNN
-F 2 "switch_cutout:SW_PUSH_6mm" H 5450 4475 50  0001 C CNN
-F 3 "~" H 5450 4475 50  0001 C CNN
-	1    5450 4275
-	1    0    0    -1
-$EndComp
-Wire Wire Line
-	5175 2675 5175 3075
-Connection ~ 5175 2675
-Wire Wire Line
-	5175 3075 5175 3475
-Wire Wire Line
-	5175 3475 5250 3475
-Connection ~ 5175 3075
-Wire Wire Line
-	5175 3475 5175 3875
-Wire Wire Line
-	5175 4675 5250 4675
-Connection ~ 5175 3475
-Wire Wire Line
-	5250 4275 5175 4275
-Connection ~ 5175 4275
-Wire Wire Line
-	5175 4275 5175 4675
-Wire Wire Line
-	5175 3875 5250 3875
-Connection ~ 5175 3875
-Wire Wire Line
-	5175 3875 5175 4275
+P 5475 3875
+F 0 "SW5" H 5475 4160 50  0000 C CNN
+F 1 "CH5" H 5475 4069 50  0000 C CNN
+F 2 "switch_cutout:SW_PUSH_6mm" H 5475 4075 50  0001 C CNN
+F 3 "~" H 5475 4075 50  0001 C CNN
+	1    5475 3875
+	1    0    0    -1
+$EndComp
+Wire Wire Line
+	5200 2275 5200 2675
+Wire Wire Line
+	5200 2675 5200 3075
+Wire Wire Line
+	5200 3075 5275 3075
+Connection ~ 5200 2675
+Wire Wire Line
+	5200 3075 5200 3475
+Wire Wire Line
+	5200 4275 5275 4275
+Connection ~ 5200 3075
+Wire Wire Line
+	5275 3875 5200 3875
+Connection ~ 5200 3875
+Wire Wire Line
+	5200 3875 5200 4275
+Wire Wire Line
+	5200 3475 5275 3475
+Connection ~ 5200 3475
+Wire Wire Line
+	5200 3475 5200 3875
 $Comp
 L Switch:SW_Push SW6
 U 1 1 62CE4BAE
-P 5450 4675
-F 0 "SW6" H 5450 4960 50  0000 C CNN
-F 1 "SYS" H 5450 4869 50  0000 C CNN
-F 2 "switch_cutout:SW_PUSH_6mm" H 5450 4875 50  0001 C CNN
-F 3 "~" H 5450 4875 50  0001 C CNN
-	1    5450 4675
+P 5475 4275
+F 0 "SW6" H 5475 4560 50  0000 C CNN
+F 1 "SYS" H 5475 4469 50  0000 C CNN
+F 2 "switch_cutout:SW_PUSH_6mm" H 5475 4475 50  0001 C CNN
+F 3 "~" H 5475 4475 50  0001 C CNN
+	1    5475 4275
 	1    0    0    -1
 $EndComp
@@
 SYS
 Wire Wire Line
-	6150 2675 5650 2675
-Entry Wire Line
-	6150 2675 6250 2775
-Wire Wire Line
-	6150 3075 5650 3075
-Entry Wire Line
-	6150 3075 6250 3175
-Wire Wire Line
-	6150 3475 5650 3475
-Entry Wire Line
-	6150 3475 6250 3575
-Wire Wire Line
-	6150 3875 5650 3875
-Entry Wire Line
-	6150 3875 6250 3975
-Wire Wire Line
-	6150 4275 5650 4275
-Entry Wire Line
-	6150 4275 6250 4375
-Wire Wire Line
-	6150 4675 5650 4675
-Entry Wire Line
-	6150 4675 6250 4775
+	6175 2275 5675 2275
+Entry Wire Line
+	6175 2275 6275 2375
+Wire Wire Line
+	6175 2675 5675 2675
+Entry Wire Line
+	6175 2675 6275 2775
+Wire Wire Line
+	6175 3075 5675 3075
+Entry Wire Line
+	6175 3075 6275 3175
+Wire Wire Line
+	6175 3475 5675 3475
+Entry Wire Line
+	6175 3475 6275 3575
+Wire Wire Line
+	6175 3875 5675 3875
+Entry Wire Line
+	6175 3875 6275 3975
+Wire Wire Line
+	6175 4275 5675 4275
+Entry Wire Line
+	6175 4275 6275 4375
 Wire Wire Line
 	7650 2675 7150 2675
@@
 Entry Wire Line
 	7650 4675 7750 4775
-Text Label 6125 2675 2    50   ~ 0
+Text Label 6150 2275 2    50   ~ 0
 SW1
-Text Label 6125 3075 2    50   ~ 0
+Text Label 6150 2675 2    50   ~ 0
 SW2
-Text Label 6125 3475 2    50   ~ 0
+Text Label 6150 3075 2    50   ~ 0
 SW3
-Text Label 6125 3875 2    50   ~ 0
+Text Label 6150 3475 2    50   ~ 0
 SW4
-Text Label 6125 4275 2    50   ~ 0
+Text Label 6150 3875 2    50   ~ 0
 SW5
-Text Label 6125 4675 2    50   ~ 0
+Text Label 6150 4275 2    50   ~ 0
 SW6
 Text Label 7625 2675 2    50   ~ 0
@@
 SYS
 Entry Bus Bus
-	6250 4950 6150 5050
+	6275 4950 6175 5050
 Entry Bus Bus
 	4550 4950 4650 5050
@@
 Connection ~ 6775 2275
 Connection ~ 6775 2675
+$Comp
+L power:GND #PWR?
+U 1 1 6630CF06
+P 5200 4425
+F 0 "#PWR?" H 5200 4175 50  0001 C CNN
+F 1 "GND" H 5205 4252 50  0000 C CNN
+F 2 "" H 5200 4425 50  0001 C CNN
+F 3 "" H 5200 4425 50  0001 C CNN
+	1    5200 4425
+	-1   0    0    -1
+$EndComp
+Wire Wire Line
+	5200 4425 5200 4275
+Connection ~ 5200 4275
+Wire Wire Line
+	3950 2475 4050 2475
+Connection ~ 4050 2475
+Wire Wire Line
+	4050 2475 4125 2475
+Wire Wire Line
+	4050 4375 4050 4650
+Wire Wire Line
+	4125 4375 4050 4375
 Wire Bus Line
 	4650 5050 7650 5050
 Wire Bus Line
-	6250 2775 6250 4950
+	6275 2375 6275 4950
 Wire Bus Line
 	7750 2375 7750 4950
