File: BulkyMIDI-32 Power Switch/BulkyMIDI-32 Power Switch.sch (KiCad schematic (older format))
At the start: 20 parts, among them J1 DC IN, J6 Power Panel, M1 Mounting, M2 Mounting, M3 Mounting, M4 Mounting, SW1 CH1, SW2 CH2, SW3 CH3, SW4 CH4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

Commit message: Power switch faceplate
Parts:
- D2: value LED -> PWR
- D3: value LED -> SYS
- J6: footprint BulkyMIDI-32:Switch_Panel -> BulkyMIDI-32:Power_Panel
Changed lines of the file:
@@
 F 0 "J6" H 10768 3975 50  0000 C CNN
 F 1 "Power Panel" H 10768 3884 50  0000 C CNN
-F 2 "BulkyMIDI-32:Switch_Panel" H 10750 2750 50  0001 C CNN
+F 2 "BulkyMIDI-32:Power_Panel" H 10750 2750 50  0001 C CNN
 F 3 "~" H 10750 2750 50  0001 C CNN
 	1    10750 2750
@@
 $EndComp
 $Comp
-L Device:LED D2
-U 1 1 664E799F
-P 4650 3425
-F 0 "D2" V 4689 3307 50  0000 R CNN
-F 1 "LED" V 4598 3307 50  0000 R CNN
-F 2 "LED_THT:LED_D3.0mm" H 4650 3425 50  0001 C CNN
-F 3 "~" H 4650 3425 50  0001 C CNN
-	1    4650 3425
-	0    -1   -1   0
-$EndComp
-$Comp
 L power:GND #PWR0119
 U 1 1 664E9624
@@
 P 5750 3425
 F 0 "D3" V 5789 3307 50  0000 R CNN
-F 1 "LED" V 5698 3307 50  0000 R CNN
+F 1 "SYS" V 5698 3307 50  0000 R CNN
 F 2 "LED_THT:LED_D3.0mm" H 5750 3425 50  0001 C CNN
 F 3 "~" H 5750 3425 50  0001 C CNN
@@
 Wire Bus Line
 	9775 1000 9775 2950
+$Comp
+L Device:LED D2
+U 1 1 664E799F
+P 4650 3425
+F 0 "D2" V 4689 3307 50  0000 R CNN
+F 1 "PWR" V 4598 3307 50  0000 R CNN
+F 2 "LED_THT:LED_D3.0mm" H 4650 3425 50  0001 C CNN
+F 3 "~" H 4650 3425 50  0001 C CNN
+	1    4650 3425
+	0    -1   -1   0
+$EndComp
 $EndSCHEMATC

Commit message: Fixes panel errors and inconsistencies
Connections:
- net +5V: now also D2.2 (A), D3.2 (A)
- net GND: no longer D2.1 (K), D3.1 (K)
- net PWR: now also D2.1 (K); no longer D2.2 (A)
- net SYS: now also D3.1 (K); no longer D3.2 (A)
Other:
- moved on the sheet: D2, D3
Changed lines of the file:
@@
 	-1   0    0    1
 $EndComp
-$Comp
-L power:GND #PWR0119
-U 1 1 664E9624
-P 4650 3575
-F 0 "#PWR0119" H 4650 3325 50  0001 C CNN
-F 1 "GND" H 4655 3402 50  0000 C CNN
-F 2 "" H 4650 3575 50  0001 C CNN
-F 3 "" H 4650 3575 50  0001 C CNN
-	1    4650 3575
-	-1   0    0    -1
-$EndComp
 Wire Wire Line
 	4650 2825 4650 2750
 Wire Wire Line
 	4650 2750 4725 2750
-Text GLabel 4475 3275 3    50   Output ~ 0
+Text GLabel 4175 3275 3    50   Output ~ 0
 PWR
 Wire Wire Line
-	4650 3125 4650 3200
-Wire Wire Line
-	4650 3200 4475 3200
-Wire Wire Line
-	4475 3200 4475 3275
-Wire Wire Line
-	4650 3200 4650 3275
-Connection ~ 4650 3200
+	4175 3200 4175 3275
 Text GLabel 10325 1950 0    50   Input ~ 0
 PWR
@@
 L Device:LED D3
 U 1 1 6655E4DA
-P 5750 3425
-F 0 "D3" V 5789 3307 50  0000 R CNN
-F 1 "SYS" V 5698 3307 50  0000 R CNN
-F 2 "LED_THT:LED_D3.0mm" H 5750 3425 50  0001 C CNN
-F 3 "~" H 5750 3425 50  0001 C CNN
-	1    5750 3425
-	0    1    -1   0
-$EndComp
-$Comp
-L power:GND #PWR0122
-U 1 1 6655E4E0
-P 5750 3575
-F 0 "#PWR0122" H 5750 3325 50  0001 C CNN
-F 1 "GND" H 5755 3402 50  0000 C CNN
-F 2 "" H 5750 3575 50  0001 C CNN
-F 3 "" H 5750 3575 50  0001 C CNN
-	1    5750 3575
-	1    0    0    -1
+P 6225 2950
+F 0 "D3" V 6264 2832 50  0000 R CNN
+F 1 "SYS" V 6173 2832 50  0000 R CNN
+F 2 "LED_THT:LED_D3.0mm" H 6225 2950 50  0001 C CNN
+F 3 "~" H 6225 2950 50  0001 C CNN
+	1    6225 2950
+	0    -1   -1   0
 $EndComp
 Wire Wire Line
@@
 Wire Wire Line
 	5750 2750 5675 2750
-Text GLabel 5925 3275 3    50   Output ~ 0
+Text GLabel 6225 3275 3    50   Output ~ 0
 SYS
-Wire Wire Line
-	5750 3125 5750 3200
-Wire Wire Line
-	5750 3200 5925 3200
-Wire Wire Line
-	5925 3200 5925 3275
-Wire Wire Line
-	5750 3200 5750 3275
-Connection ~ 5750 3200
 NoConn ~ 5675 2550
 NoConn ~ 5675 2650
@@
 Wire Bus Line
 	8000 1000 9775 1000
-Wire Bus Line
-	8000 1000 8000 2350
-Wire Bus Line
-	4275 1000 4275 2450
-Wire Bus Line
-	2525 1000 2525 4000
-Wire Bus Line
-	9775 1000 9775 2950
 $Comp
 L Device:LED D2
 U 1 1 664E799F
-P 4650 3425
-F 0 "D2" V 4689 3307 50  0000 R CNN
-F 1 "PWR" V 4598 3307 50  0000 R CNN
-F 2 "LED_THT:LED_D3.0mm" H 4650 3425 50  0001 C CNN
-F 3 "~" H 4650 3425 50  0001 C CNN
-	1    4650 3425
-	0    -1   -1   0
-$EndComp
+P 4175 2950
+F 0 "D2" V 4214 2832 50  0000 R CNN
+F 1 "PWR" V 4123 2832 50  0000 R CNN
+F 2 "LED_THT:LED_D3.0mm" H 4175 2950 50  0001 C CNN
+F 3 "~" H 4175 2950 50  0001 C CNN
+	1    4175 2950
+	0    1    -1   0
+$EndComp
+Wire Wire Line
+	4650 3125 4650 3200
+Wire Wire Line
+	4175 3100 4175 3200
+Connection ~ 4175 3200
+Wire Wire Line
+	4175 3200 4650 3200
+$Comp
+L power:+5V #PWR?
+U 1 1 663248CA
+P 4175 2800
+F 0 "#PWR?" H 4175 2650 50  0001 C CNN
+F 1 "+5V" H 4175 2950 50  0000 C CNN
+F 2 "" H 4175 2800 50  0001 C CNN
+F 3 "" H 4175 2800 50  0001 C CNN
+	1    4175 2800
+	1    0    0    -1
+$EndComp
+$Comp
+L power:+5V #PWR?
+U 1 1 6632A808
+P 6225 2800
+F 0 "#PWR?" H 6225 2650 50  0001 C CNN
+F 1 "+5V" H 6225 2950 50  0000 C CNN
+F 2 "" H 6225 2800 50  0001 C CNN
+F 3 "" H 6225 2800 50  0001 C CNN
+	1    6225 2800
+	1    0    0    -1
+$EndComp
+Wire Wire Line
+	5750 3125 5750 3200
+Wire Wire Line
+	6225 3200 5750 3200
+Wire Wire Line
+	6225 3100 6225 3200
+Wire Wire Line
+	6225 3275 6225 3200
+Connection ~ 6225 3200
+Wire Bus Line
+	8000 1000 8000 2350
+Wire Bus Line
+	4275 1000 4275 2450
+Wire Bus Line
+	2525 1000 2525 4000
+Wire Bus Line
+	9775 1000 9775 2950
 $EndSCHEMATC

Commit message: Updated Power Switch to incorporate changes
Connections:
- no-connect marks 8 -> 7
Changed lines of the file:
@@
 	1    0    0    -1
 $EndComp
-NoConn ~ 6600 150
 $Comp
 L BulkyMIDI:DC_5V SYM1
