File: BulkyMIDI-32 Power Switch/BulkyMIDI-32 Power Switch.kicad_sch (KiCad schematic)
At the start: 20 parts, among them J1 DC IN, J6 Power Panel, M1 Mounting, M2 Mounting, M3 Mounting, M4 Mounting, SW1 CH1, SW2 CH2, SW3 CH3, SW4 CH4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

Commit message: Updated Power Switch
Parts:
- added F1: Fuse, BulkyMIDI-32:Fuseholder5x20_horiz_SemiClosed_Casing10x25mm, symbol Device:Fuse
- M1, M2, M3, M4: footprint mounting:M3 -> mounting:M3_pin; symbol mounting:Mounting -> mounting:Mounting_Pin
Connections:
- net GND: now also M1.1, M2.1, M3.1, M4.1
- net VIN: now also F1.1; no longer D1.2 (A)
- new net: D1.2 (A), F1.2
Other:
- moved on the sheet: C6, D1
